File: eagle/Ignition Board/Ignition_Board.sch (EAGLE design)
At the start: 21 parts, among them IC1 INVERT GATES, IC2 OPTOISOLATOR, Q1 NMOSFET

Commit message: Pushed latest ignition board, power board, and updated launch-tower library files. Also changed directory structure.
Parts:
- removed JP1: 5MM screw, SparkFun:M025MM
- removed ZD1: DIODE-ZENERPTH, SparkFun:DIODE-ZENERPTH
- added BATT-IN, BATT-OUT: 5MM screw, SparkFun:M025MM
- added C3, C4: (no value), rcl_custom:C-EU0805-B-NOSILK
- added C5: 10, rcl_custom:C-EU0805-B-NOSILK
- added C6: 0.01, rcl_custom:C-EU0805-B-NOSILK
- added R8: 100, rcl_custom:R-US_0805-B-NOSILK
- added R9: 0k, rcl_custom:R-US_0805-B-NOSILK
- added U$2, U$3, U$4, U$5: #4-BARE_MOUNTING_HOLE/.300, mount:#4-BARE_MOUNTING_HOLE/.300
- added U$6: BATTERY, launch-tower:BATTERY
- R1: value (none) -> 4.7k
- R2: value (none) -> PICK ME
Connections:
- net N-NOT1 renamed N$15
- removed net VFIRE-IN: JP1.2, L1.SW2
- removed net VFIRE-OUT: JP1.1, L1.SW1
- removed net VROCKET: JP3.1, ZD1.A
- new net GND-BATT: BATT-IN.2, BATT-OUT.1, U$6.GND
- new net N$11: C3.2, U$1.+V
- new net N$4: JP3.1, R8.2
- new net ROCKET-READY: R1.2, R2.2, R8.1, ZD2.C
- new net VCC-BATT: BATT-IN.1, BATT-OUT.2, L1.SW1, L1.SW2, U$6.VCC
- new net VDD: C3.1, C4.1, D6.C, L1.COUT, R3.2, R9.2
- net GND: now also C5.2, C6.2
- net N$12: now also C5.1, C6.1, R9.1; no longer D6.C, IC1.VCC, L1.COUT, R3.2, U$1.+V
- net N$8: now also C4.2, IC1.VCC; no longer R1.2, R2.2, ZD1.C, ZD2.C
Other:
- note added: "ROCKET-READY is a 5V (@ 50 mA max)"
- note added: "VSAMPLE is the shore power connector"
- note added: "signal from the rocket."
- note added: "to the rocket."
- moved on the sheet: C1, C2, D5, D6, IC1, IC2, JP2, JP3, L1, Q1, R1, R2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
