File: eagle/Ignition Board/Launch_Tower_Ignition_Board_v5-0.sch (EAGLE design)
At the start: 32 parts, among them IC1 INVERT GATES, IC2 OPTOISOLATOR, Q1 NMOSFET

Commit message: Richard Witherspoon - latest version of LTC boards
Parts:
- removed BATT-OUT: 5MM screw, SparkFun:M025MM
- removed D6: (no value), SparkFun:DIODEPTH
- removed L1: RELAY, launch-tower:RELAY
- removed R2: PICK ME, rcl_custom:R-US_0805-B-NOSILK
- removed ZD2: DIODE-ZENERPTH, SparkFun:DIODE-ZENERPTH
- added C7: NP, SparkFun:CAPPTH
- added CHARGER-IN, IGNITION: 5MM screw, SparkFun:M025MM
- added D3: 1N4148/1N4448, SparkFun:DIODEPTH
- added JP1, JP5: JUMPER-3PTH, SparkFun:JUMPER-3PTH
- added LED1: (no value), SparkFun:LED-FKIT-1206
- added R10: NP, SparkFun:RESISTORPTH-1/4W
- added R11: 0k, rcl_custom:R-US_0805-B-NOSILK
- added U1: SN65220DBV, sn65220:SN65220DBV
- C1: value (none) -> .1uF
- C2: value (none) -> 1uF
- C3, C4: value (none) -> 0.1uF
- D5: value (none) -> 1N4148/1N4448
- R1: value 4.7k -> 10k
- R3, R4, R7: value (none) -> 10k
- R5: value (none) -> 2.6k
- R6: value (none) -> 1M
- R8: value 100 -> 350
- R9: value 0k -> 0
- U$6: value BATTERY -> RELAY-2; device launch-tower:BATTERY -> launch-tower:RELAY-2
Connections:
- removed net N$8: C4.2, IC1.VCC
- new net BATT-CHARG-RELAY: CHARGER-IN.1, U$6.NC
- new net N$2: LED1.A, R11.1
- new net VCC-IGNITION: IGNITION.1, U$6.NO
- net GND: now also C3.2, C4.2, C7.2, IC1.5A, IC1.6A, LED1.C, U1.GND, U1.GND2; no longer ZD2.A
- net GND-BATT: now also CHARGER-IN.2, IGNITION.2; no longer BATT-OUT.1, U$6.GND
- net N$1: now also JP1.2; no longer IC1.2Y
- net N$11: now also IC1.1Y, JP5.1; no longer C3.2, U$1.+V
- net N$12: now also R11.2
- net N$13: now also R10.1
- net N$15: now also C7.1, R10.2
- net N$5: now also JP5.2; no longer IC1.1Y
- net N$6: now also IC1.2Y, JP1.3; no longer IC2.A, R2.1
- net N$7: now also U1.B
- net N$9: now also D3.A, U$6.CIN; no longer D6.A, L1.CIN
- net ROCKET-READY: now also IC2.A, U1.A; no longer R2.2, ZD2.C
- net VCC-BATT: now also U$6.SOURCE; no longer BATT-OUT.2, L1.SW1, L1.SW2, U$6.VCC
- net VDD: now also D3.C, IC1.VCC, JP1.1, JP5.3, U$1.+V, U$6.COUT; no longer D6.C, L1.COUT
Other:
- note added: "0.5A 1s || 1A 1 ms || 4A 1μs"
- note added: "5 second charge time"
- note added: "Capacitor @ supply voltage @ 5T or 5 x RC"
- note added: "Chnage to 1 time constant"
- note added: "DC Input or Output Voltage --> 0V to VCC"
- note added: "Full voltage time (secs) = 5 (R x C)"
- note added: "Gate Input Voltage --> up to 5.5v"
- note added: "Input Voltage --> 1.2v - 1.5v"
- note added: "Note: Want small capacitor for fast discharge"
- note added: "OUT"
- note added: "P/N: 1N4148/1N4448"
- note added: "P/N: 4N35-300E"
- note added: "P/N: CD74HC14M96"
- note added: "P/N: SN74LVC1G08"
- note added: "R1 (r4) = 10k"
- note added: "R1 = ( (R2 x Vin) / (Vout) ) - R2"
- note added: "R2 (r5) = 10k / ( (24v - 5v) - 1 ) = 2.6K"
- note added: "R2 = ( R1 / (Vin / Vout) - 1 )"
- note added: "R4: I=V/R = 5v/10,000 Ohm = 0.0005A = 0.5mA"
- note added: "T = R (Ohms) x C (farads)"
- note added: "Time constant for charging"
- note added: "Vout / Vin = R2 / (R1 + R2)"
- note added: "Vout = (Z2 / (Z1 + z2) ) x Vin"
- note added: "http://www.electronics-tutorials.ws/rc/rc_1.html"
- note added: "to the rocket (CALCED @ 24v)."
- note added: "~ 4.7M resistor"
- note removed: "to the rocket."
- moved on the sheet: BATT-IN, C1, C2, C3, C4, D5, IC1, Q1, R1, R4, R5, R6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
