File: eagle/Power Interface Board/Launch_Tower_Power_Interface_Board_v1-1.brd (EAGLE design)
At the start: 105.1 x 71.1 mm, 35 parts

Commit message: Richard Witherspoon - latest version of LTC boards
Parts:
- added LTC-OUT1: (no value), SparkFun:SCREWTERMINAL-5MM-2
- moved 5V-OUT-1 18.2 mm to (92.7, 66.0), turned to 180 degrees
- moved 5V-OUT-2 15.3 mm to (85.1, 66.0), turned to 180 degrees
- moved 19V-OUT-1 1.27 mm to (97.8, 14.0)
- moved 19V-OUT-2 1.27 mm to (97.8, 25.4)
- moved JP1 1.27 mm to (80.0, 14.0)
- moved LTC-OUT 1.27 mm to (97.8, 36.8)
- moved RELAY-19V-2 1.27 mm to (71.1, 7.62)
- moved 19V-DC/DC-IN 1.27 mm to (55.9, 7.62)
- moved R1 1.27 mm to (40.6, 49.5)
- moved R2 1.27 mm to (40.6, 41.9)
- moved R3 1.27 mm to (40.6, 30.5)
- moved R4 1.27 mm to (40.6, 26.7)
- moved R7 1.27 mm to (40.6, 45.7)
- moved R8 1.27 mm to (40.6, 38.1)
- moved R9 1.27 mm to (40.6, 34.3)
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Connections:
- net N$7 renamed VBAT
- removed net N$26: DC1.2, LTC-OUT.2, R2.P$1, SWITCH.2, TO-19V-DC/DC.1
- new net VLTC: DC1.2, LTC-OUT.2, LTC-OUT1.2, R2.P$1, SWITCH.2, TO-19V-DC/DC.1
- net GND: now also LTC-OUT1.1
Routing:
- net VLTC: track 0.00 -> 206.0 mm, vias 0 -> 3
- net N$26: track 193.2 -> 0.00 mm, vias 3 -> 0
- net N$17: track 109.2 -> 96.5 mm, vias 4 -> 1
- net GND: track 113.8 -> 118.8 mm, vias 15 -> 16
- net N$12: track 110.5 -> 113.1 mm, vias 2 -> 4
- net N$15: vias 3 -> 2
Other:
- board size 105.1 x 71.1 mm -> 105.4 x 71.1 mm
