File: eagle/Power Interface Board/Launch_Tower_Power_Interface_Board_v1-1.sch (EAGLE design)
At the start: 35 parts

Commit message: Richard Witherspoon - latest version of LTC boards
Parts:
- added LTC-OUT1: (no value), SparkFun:M025MM
Connections:
- net N$7 renamed VBAT
- removed net N$26: DC1.+VIN, LTC-OUT.2, R2.1, SWITCH.2, TO-19V-DC/DC.1
- new net VLTC: DC1.+VIN, LTC-OUT.2, LTC-OUT1.2, R2.1, SWITCH.2, TO-19V-DC/DC.1
- net GND: now also LTC-OUT1.1
Other:
- moved on the sheet: LED-BATTERY-IN, LED-SOLAR-IN, R1, R7
