File: ltc3/kicad/BBB_Cape.sch (KiCad schematic (older format))
At the start: 11 parts

Commit message: Minor progress on LTC3 schematics.
Parts:
- removed R? (x2): 4.7k, ~, symbol R
- removed SW?: DIPS_03, symbol DIPS_03
- removed U?: 24C256, symbol 24C256
- added JP?: WP DISABLE, ~, symbol JUMPER
- added R? (x2): 5.6k, ~, symbol R
- added U?: LTC2991, symbol LTC2991
- added U?: 24C256, ~, symbol 24C256
- R? (x2): value 4.7k -> 5.6k
Connections:
- net labels added: I2C1_SCL, I2C1_SDA
- wire segments 60 -> 62
Other:
- note added: "Cape EEPROM\nIC2 addr 0x54"
- note added: "Voltage & Temp Sensor\nI2C addr 0x90"
- moved on the sheet: C?, R?
