File: ltc3/kicad/triggers.sch (KiCad schematic (older format))
At the start: 16 parts, among them K1 RELAY_SPDT, K2 RELAY_SPDT, K3 RELAY_SPDT, K4 RELAY_SPDT, Q1 PMV45EN, Q2 PMV45EN, Q3 PMV45EN, Q4 PMV45EN

Commit message: Fixed mistakes in triggers schematic; misc. clean-up.
Parts:
- added D1, D2, D3, D4: 1N4001, ~, symbol DIODE
- added K5, K6, K7, K8: EURO 3POS, symbol CONN_3
Connections:
- net labels added: VCC_5V
- wire segments 38 -> 70
Other:
- note removed: "TODO:\nThree-conductor\njacks go here!"
- moved on the sheet: F1, F2, F3, F4, R10, R7, R8, R9

Commit message: Fixed incorrect FET symbol on LTC3 ext. triggers schematic.
Parts:
- removed Q1, Q2, Q3, Q4: PMV45EN, SOT23, symbol MOSFET_N
- added Q? (x4): PMV45EN, ~, symbol MOSFET_N
Changed lines of the file:
@@
 Sheet 6 6
 Title "LTC3 External Triggers"
-Date "2 apr 2015"
+Date "3 apr 2015"
 Rev "1"
 Comp "Portland State Aerospace Society <http://psas.pdx.edu/>"
@@
 $EndComp
 $Comp
-L MOSFET_N Q1
-U 1 1 551C7F19
-P 3250 2700
-F 0 "Q1" H 3260 2870 60  0000 R CNN
-F 1 "PMV45EN" H 3260 2550 60  0000 R CNN
-F 2 "SOT23" H 3250 2700 60  0001 C CNN
-F 3 "~" H 3250 2700 60  0000 C CNN
-	1    3250 2700
-	1    0    0    -1
-$EndComp
-$Comp
 L GND #PWR8
 U 1 1 551C7F4B
@@
 $EndComp
 $Comp
-L MOSFET_N Q2
-U 1 1 551C82F4
-P 3250 3650
-F 0 "Q2" H 3260 3820 60  0000 R CNN
-F 1 "PMV45EN" H 3260 3500 60  0000 R CNN
-F 2 "SOT23" H 3250 3650 60  0001 C CNN
-F 3 "~" H 3250 3650 60  0000 C CNN
-	1    3250 3650
-	1    0    0    -1
-$EndComp
-$Comp
 L RELAY_SPDT K4
 U 1 1 551C8300
@@
 $EndComp
 $Comp
-L MOSFET_N Q3
-U 1 1 551CDD96
-P 3250 4650
-F 0 "Q3" H 3260 4820 60  0000 R CNN
-F 1 "PMV45EN" H 3260 4500 60  0000 R CNN
-F 2 "SOT23" H 3250 4650 60  0001 C CNN
-F 3 "~" H 3250 4650 60  0000 C CNN
-	1    3250 4650
-	1    0    0    -1
-$EndComp
-$Comp
 L GND #PWR10
 U 1 1 551CDD9C
@@
 $EndComp
 $Comp
-L MOSFET_N Q4
-U 1 1 551CDDFA
-P 3250 5650
-F 0 "Q4" H 3260 5820 60  0000 R CNN
-F 1 "PMV45EN" H 3260 5500 60  0000 R CNN
-F 2 "SOT23" H 3250 5650 60  0001 C CNN
-F 3 "~" H 3250 5650 60  0000 C CNN
-	1    3250 5650
-	1    0    0    -1
-$EndComp
-$Comp
 L GND #PWR11
 U 1 1 551CDE00
@@
 Wire Wire Line
 	7450 2050 8450 2050
+$Comp
+L MOSFET_N Q?
+U 1 1 551E1A59
+P 3250 2700
+F 0 "Q?" H 3260 2870 60  0000 R CNN
+F 1 "PMV45EN" H 3260 2550 60  0000 R CNN
+F 2 "~" H 3250 2700 60  0000 C CNN
+F 3 "~" H 3250 2700 60  0000 C CNN
+	1    3250 2700
+	1    0    0    -1
+$EndComp
+$Comp
+L MOSFET_N Q?
+U 1 1 551E1A83
+P 3250 3650
+F 0 "Q?" H 3260 3820 60  0000 R CNN
+F 1 "PMV45EN" H 3260 3500 60  0000 R CNN
+F 2 "~" H 3250 3650 60  0000 C CNN
+F 3 "~" H 3250 3650 60  0000 C CNN
+	1    3250 3650
+	1    0    0    -1
+$EndComp
+$Comp
+L MOSFET_N Q?
+U 1 1 551E1A89
+P 3250 4650
+F 0 "Q?" H 3260 4820 60  0000 R CNN
+F 1 "PMV45EN" H 3260 4500 60  0000 R CNN
+F 2 "~" H 3250 4650 60  0000 C CNN
+F 3 "~" H 3250 4650 60  0000 C CNN
+	1    3250 4650
+	1    0    0    -1
+$EndComp
+$Comp
+L MOSFET_N Q?
+U 1 1 551E1A8F
+P 3250 5650
+F 0 "Q?" H 3260 5820 60  0000 R CNN
+F 1 "PMV45EN" H 3260 5500 60  0000 R CNN
+F 2 "~" H 3250 5650 60  0000 C CNN
+F 3 "~" H 3250 5650 60  0000 C CNN
+	1    3250 5650
+	1    0    0    -1
+$EndComp
 $EndSCHEMATC

Commit message: Incremental progress on LTC3 design spec, schematic.
Parts:
- gave numbers to parts that had none: 4
Changed lines of the file:
@@
 Sheet 6 6
 Title "LTC3 External Triggers"
-Date "3 apr 2015"
+Date "4 apr 2015"
 Rev "1"
 Comp "Portland State Aerospace Society <http://psas.pdx.edu/>"
@@
 	7450 2050 8450 2050
 $Comp
-L MOSFET_N Q?
+L MOSFET_N Q1
 U 1 1 551E1A59
 P 3250 2700
-F 0 "Q?" H 3260 2870 60  0000 R CNN
+F 0 "Q1" H 3260 2870 60  0000 R CNN
 F 1 "PMV45EN" H 3260 2550 60  0000 R CNN
 F 2 "~" H 3250 2700 60  0000 C CNN
@@
 $EndComp
 $Comp
-L MOSFET_N Q?
+L MOSFET_N Q2
 U 1 1 551E1A83
 P 3250 3650
-F 0 "Q?" H 3260 3820 60  0000 R CNN
+F 0 "Q2" H 3260 3820 60  0000 R CNN
 F 1 "PMV45EN" H 3260 3500 60  0000 R CNN
 F 2 "~" H 3250 3650 60  0000 C CNN
@@
 $EndComp
 $Comp
-L MOSFET_N Q?
+L MOSFET_N Q3
 U 1 1 551E1A89
 P 3250 4650
-F 0 "Q?" H 3260 4820 60  0000 R CNN
+F 0 "Q3" H 3260 4820 60  0000 R CNN
 F 1 "PMV45EN" H 3260 4500 60  0000 R CNN
 F 2 "~" H 3250 4650 60  0000 C CNN
@@
 $EndComp
 $Comp
-L MOSFET_N Q?
+L MOSFET_N Q4
 U 1 1 551E1A8F
 P 3250 5650
-F 0 "Q?" H 3260 5820 60  0000 R CNN
+F 0 "Q4" H 3260 5820 60  0000 R CNN
 F 1 "PMV45EN" H 3260 5500 60  0000 R CNN
 F 2 "~" H 3250 5650 60  0000 C CNN
