File: ltc3/kicad/external_device_support.sch (KiCad schematic (older format))
At the start: 44 parts, among them IC1 TLP3542, IC2 TLP3542, IC3 TLP3542, IC4 TLP3542, IC5 TLP3542, IC6 TLP3542, IC7 TLP3542, IC8 TLP3542, P1 CONN_2, P2 CONN_2, P3 CONN_2, P4 CONN_2, P5 CONN_2, P6 CONN_2, P7 CONN_2, P8 CONN_2, Q1 PMV45EN, Q2 PMV45EN, Q3 PMV45EN, Q4 PMV45EN, Q5 PMV45EN, Q6 PMV45EN, Q7 PMV45EN, Q8 PMV45EN

Commit message: Updated design spec; schematic. Completed "External Device Support" section of design spec. Replaced fuses with PTC devices in external device support schematic.
Parts:
- removed F2, F4, F6, F8: 2 A, Slow, ~, symbol FUSE
- removed F3, F5, F7: 100 mA, ~, symbol FUSE
- added PTC1, PTC3, PTC5, PTC7: 06R120B, ~, symbol THERMISTOR
- added PTC2, PTC4, PTC6: 06R075B, ~, symbol THERMISTOR
Changed lines of the file:
@@
 	1    0    0    -1
-$EndComp
-$Comp
-L FUSE F2
-U 1 1 5522C598
-P 4250 2500
-F 0 "F2" H 4350 2550 40  0000 C CNN
-F 1 "2 A, Slow" H 4250 2375 40  0000 C CNN
-F 2 "~" H 4250 2500 60  0000 C CNN
-F 3 "~" H 4250 2500 60  0000 C CNN
-	1    4250 2500
-	0    1    1    0
 $EndComp
 Text HLabel 2400 3450 0    60   Input ~ 0
@@
 	1    0    0    -1
 $EndComp
-$Comp
-L FUSE F4
-U 1 1 55252F1F
-P 7750 2500
-F 0 "F4" H 7850 2550 40  0000 C CNN
-F 1 "2 A, Slow" H 7750 2375 40  0000 C CNN
-F 2 "~" H 7750 2500 60  0000 C CNN
-F 3 "~" H 7750 2500 60  0000 C CNN
-	1    7750 2500
-	0    1    1    0
-$EndComp
 Text HLabel 5900 3450 0    60   Input ~ 0
 GPIO_EXT_PWR_2
@@
 	1    0    0    -1
 $EndComp
-$Comp
-L FUSE F6
-U 1 1 55252F61
-P 11250 2500
-F 0 "F6" H 11350 2550 40  0000 C CNN
-F 1 "2 A, Slow" H 11250 2375 40  0000 C CNN
-F 2 "~" H 11250 2500 60  0000 C CNN
-F 3 "~" H 11250 2500 60  0000 C CNN
-	1    11250 2500
-	0    1    1    0
-$EndComp
 Text HLabel 9400 3450 0    60   Input ~ 0
 GPIO_EXT_PWR_3
@@
 	1    13150 3850
 	1    0    0    -1
-$EndComp
-$Comp
-L FUSE F8
-U 1 1 55252FA3
-P 14750 2500
-F 0 "F8" H 14850 2550 40  0000 C CNN
-F 1 "2 A, Slow" H 14750 2375 40  0000 C CNN
-F 2 "~" H 14750 2500 60  0000 C CNN
-F 3 "~" H 14750 2500 60  0000 C CNN
-	1    14750 2500
-	0    1    1    0
 $EndComp
 Text HLabel 12900 3450 0    60   Input ~ 0
@@
 	1    0    0    -1
 $EndComp
-$Comp
-L FUSE F3
-U 1 1 55253251
-P 7350 6350
-F 0 "F3" H 7450 6400 40  0000 C CNN
-F 1 "100 mA" H 7350 6225 40  0000 C CNN
-F 2 "~" H 7350 6350 60  0000 C CNN
-F 3 "~" H 7350 6350 60  0000 C CNN
-	1    7350 6350
-	0    1    1    0
-$EndComp
 Text HLabel 5900 7550 0    60   Input ~ 0
 GPIO_EXT_TRIG_2
@@
 	1    0    0    -1
 $EndComp
-$Comp
-L FUSE F5
-U 1 1 552532A4
-P 10850 6350
-F 0 "F5" H 10950 6400 40  0000 C CNN
-F 1 "100 mA" H 10850 6225 40  0000 C CNN
-F 2 "~" H 10850 6350 60  0000 C CNN
-F 3 "~" H 10850 6350 60  0000 C CNN
-	1    10850 6350
-	0    1    1    0
-$EndComp
 Text HLabel 9400 7550 0    60   Input ~ 0
 GPIO_EXT_TRIG_3
@@
 	1    13150 7950
 	1    0    0    -1
-$EndComp
-$Comp
-L FUSE F7
-U 1 1 552532F7
-P 14350 6350
-F 0 "F7" H 14450 6400 40  0000 C CNN
-F 1 "100 mA" H 14350 6225 40  0000 C CNN
-F 2 "~" H 14350 6350 60  0000 C CNN
-F 3 "~" H 14350 6350 60  0000 C CNN
-	1    14350 6350
-	0    1    1    0
 $EndComp
 Text HLabel 12900 7550 0    60   Input ~ 0
@@
 Text Notes 1400 4750 0    100  ~ 0
 External Device Power
+$Comp
+L THERMISTOR PTC1
+U 1 1 5524D181
+P 4250 2500
+F 0 "PTC1" V 4350 2550 50  0000 C CNN
+F 1 "06R120B" V 4150 2500 50  0000 C CNN
+F 2 "~" H 4250 2500 60  0000 C CNN
+F 3 "~" H 4250 2500 60  0000 C CNN
+	1    4250 2500
+	1    0    0    -1
+$EndComp
+$Comp
+L THERMISTOR PTC3
+U 1 1 5524D1A4
+P 7750 2500
+F 0 "PTC3" V 7850 2550 50  0000 C CNN
+F 1 "06R120B" V 7650 2500 50  0000 C CNN
+F 2 "~" H 7750 2500 60  0000 C CNN
+F 3 "~" H 7750 2500 60  0000 C CNN
+	1    7750 2500
+	1    0    0    -1
+$EndComp
+$Comp
+L THERMISTOR PTC5
+U 1 1 5524D1B4
+P 11250 2500
+F 0 "PTC5" V 11350 2550 50  0000 C CNN
+F 1 "06R120B" V 11150 2500 50  0000 C CNN
+F 2 "~" H 11250 2500 60  0000 C CNN
+F 3 "~" H 11250 2500 60  0000 C CNN
+	1    11250 2500
+	1    0    0    -1
+$EndComp
+$Comp
+L THERMISTOR PTC7
+U 1 1 5524D1BA
+P 14750 2500
+F 0 "PTC7" V 14850 2550 50  0000 C CNN
+F 1 "06R120B" V 14650 2500 50  0000 C CNN
+F 2 "~" H 14750 2500 60  0000 C CNN
+F 3 "~" H 14750 2500 60  0000 C CNN
+	1    14750 2500
+	1    0    0    -1
+$EndComp
+$Comp
+L THERMISTOR PTC2
+U 1 1 5524D1C0
+P 7350 6350
+F 0 "PTC2" V 7450 6400 50  0000 C CNN
+F 1 "06R075B" V 7250 6350 50  0000 C CNN
+F 2 "~" H 7350 6350 60  0000 C CNN
+F 3 "~" H 7350 6350 60  0000 C CNN
+	1    7350 6350
+	1    0    0    -1
+$EndComp
+$Comp
+L THERMISTOR PTC4
+U 1 1 5524D1DC
+P 10850 6350
+F 0 "PTC4" V 10950 6400 50  0000 C CNN
+F 1 "06R075B" V 10750 6350 50  0000 C CNN
+F 2 "~" H 10850 6350 60  0000 C CNN
+F 3 "~" H 10850 6350 60  0000 C CNN
+	1    10850 6350
+	1    0    0    -1
+$EndComp
+$Comp
+L THERMISTOR PTC6
+U 1 1 5524D1E2
+P 14350 6350
+F 0 "PTC6" V 14450 6400 50  0000 C CNN
+F 1 "06R075B" V 14250 6350 50  0000 C CNN
+F 2 "~" H 14350 6350 60  0000 C CNN
+F 3 "~" H 14350 6350 60  0000 C CNN
+	1    14350 6350
+	1    0    0    -1
+$EndComp
 $EndSCHEMATC
