File: ltc3/kicad/rocket_interface.sch (KiCad schematic (older format))
At the start: 37 parts

Commit message: LTC3: Misc. edits to rocket umbilical schematic.
Parts:
- removed K?: RELAY_SPDT, symbol RELAY_SPDT
- removed P?: TEST-LEAD-ROCKETREADY, symbol CONN_01X02
- removed P?: TEST-LEAD-VSAMPLE, symbol CONN_01X02
- removed P?: CHARGER-IN, symbol CONN_01X02
- added K401: RELAY_1C, symbol RELAY_1C
- gave numbers to parts that had none: 28
Connections:
- net +5V: now also D401.2 (A), Q401.3 (D), K401.85 (COIL2); no longer D401.1 (K)
- net GND: now also U402.5; no longer U402.12, U402.13
- net IGNITION: now also K401.87 (NO)
- net IGN_BATT: now also K401.30 (COM)
- net at R412.2: now also U402.12; no longer U402.10
- net at U402.2: now also R404.1, U403.1 (A)
- net at R405.1, U403.2 (B): now also U402.4
- net at C404.1, C405.1, R408.1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: now also U402.11; no longer U402.5
- new net: D401.1 (K), K401.86 (COIL1)
- new net: U402.10, U402.13, U402.9
Other:
- note added: "TODO:\n* Select appropriate component values.\n* Move TVS upstream of voltage dividers."
- note removed: "TODO:\n* Select appropriate component values.\n\nQUESTIONS:\n* Keep the "test" jumpers?\n* Do we need to integrate a charger for the ignition\n battery?\n* Where's the launch/ignition signal?\n* What's the purpose of the TVS on the\n input signals? It clamps at 7V, more than enough\n to look like a genuine high input.\n* What's the purpose of the extra resistor and cap.\n in the delay stage? Post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"
- moved on the sheet: D401, P402, P403, R404, R405
