File: ltc3/kicad/_saved_battery_balance.sch (KiCad schematic (older format))
At the start: 75 parts, among them P301 CONN_BATT_MAIN, P302 CONN_BATT_SENSE, P303 S2BPHKS, Q301 NDS9407, Q302 MMBT3904, Q303 SUM110P08-11, Q304 SUM110P08-11, Q305 SUM110P08-11, Q306 SUM110P08-11, U301 LTC2990, U302 BQ77PL900

Commit message: Selected Footprints
Parts:
- P301, P302, P303: footprint (none) -> Pin_Headers:Pin_Header_Straight_1x02
Changed lines of the file:
@@
 F 0 "P302" H 9600 7500 50  0000 C CNN
 F 1 "CONN_BATT_SENSE" V 9700 7050 50  0000 C CNN
-F 2 "" H 9600 7050 60  0001 C CNN
+F 2 "Pin_Headers:Pin_Header_Straight_1x02" H 9600 7050 60  0001 C CNN
 F 3 "" H 9600 7050 60  0000 C CNN
 	1    9600 7050
@@
 F 0 "P301" H 10350 5950 50  0000 C CNN
 F 1 "CONN_BATT_MAIN" V 10450 5800 50  0000 C CNN
-F 2 "" H 10350 5800 60  0001 C CNN
+F 2 "Pin_Headers:Pin_Header_Straight_1x02" H 10350 5800 60  0001 C CNN
 F 3 "" H 10350 5800 60  0000 C CNN
 	1    10350 5800
@@
 F 0 "P303" H 2600 7550 50  0000 C CNN
 F 1 "S2BPHKS" V 2700 7400 50  0000 C CNN
-F 2 "" H 2600 7400 60  0001 C CNN
+F 2 "Pin_Headers:Pin_Header_Straight_1x02" H 2600 7400 60  0001 C CNN
 F 3 "" H 2600 7400 60  0000 C CNN
 	1    2600 7400
