File: ltc3/kicad/_saved_power_in_charge_controller.sch (KiCad schematic (older format))
At the start: 112 parts, among them P201 PV_IN, P202 LAB_IN, P203 S2BPHKS, Q201 BSC028N06NS, Q202 BSC028N06NS, Q203 BSC028N06NS, Q204 BSC028N06NS, Q205 ZVN4525E6, Q206 ZVP3310F, Q207 MMBT5550L, U201 PI2127, U202 PI2127, U203 LTC2990, U204 LT8490

Commit message: Finished footprint assignment.
Parts:
- D203, D204, D205: footprint Capacitors_ThroughHole:C_Radial_D10_L20_P2.5 -> Choke_Axial_ThroughHole:Choke_Horizontal_RM10mm
- P201: footprint (none) -> Connectors_Molex:Molex_KK_6410-02
- P202: footprint (none) -> Connectors_Molex:Molex_KK_6410-03
Changed lines of the file:
@@
 F 0 "D204" H 7400 9600 50  0000 C CNN
 F 1 "LED" H 7400 9400 50  0000 C CNN
-F 2 "Capacitors_ThroughHole:C_Radial_D10_L20_P2.5" H 7400 9500 60  0001 C CNN
+F 2 "Choke_Axial_ThroughHole:Choke_Horizontal_RM10mm" H 7400 9500 60  0001 C CNN
 F 3 "" H 7400 9500 60  0000 C CNN
 	1    7400 9500
@@
 F 0 "D205" H 7850 9600 50  0000 C CNN
 F 1 "LED" H 7850 9400 50  0000 C CNN
-F 2 "Capacitors_ThroughHole:C_Radial_D10_L20_P2.5" H 7850 9500 60  0001 C CNN
+F 2 "Choke_Axial_ThroughHole:Choke_Horizontal_RM10mm" H 7850 9500 60  0001 C CNN
 F 3 "" H 7850 9500 60  0000 C CNN
 	1    7850 9500
@@
 F 0 "P201" H 800 900 50  0000 C CNN
 F 1 "PV_IN" V 900 1050 50  0000 C CNN
-F 2 "" H 800 1050 60  0001 C CNN
+F 2 "Connectors_Molex:Molex_KK_6410-02" H 800 1050 60  0001 C CNN
 F 3 "" H 800 1050 60  0000 C CNN
 	1    800  1050
@@
 F 0 "P202" H 800 2650 50  0000 C CNN
 F 1 "LAB_IN" V 900 2850 50  0000 C CNN
-F 2 "" H 800 2800 60  0001 C CNN
+F 2 "Connectors_Molex:Molex_KK_6410-03" H 800 2800 60  0001 C CNN
 F 3 "" H 800 2800 60  0000 C CNN
 	1    800  2800
@@
 F 0 "D203" H 14400 5900 50  0000 C CNN
 F 1 "1N4743A" H 14400 6100 50  0000 C CNN
-F 2 "Capacitors_ThroughHole:C_Radial_D10_L20_P2.5" H 14400 6000 60  0001 C CNN
+F 2 "Choke_Axial_ThroughHole:Choke_Horizontal_RM10mm" H 14400 6000 60  0001 C CNN
 F 3 "" H 14400 6000 60  0000 C CNN
 F 4 "13V" H 14400 6200 50  0000 C CIN "Note"
