File: ltc3/kicad/_saved_rocket_interface.sch (KiCad schematic (older format))
At the start: 68 parts, among them IC601 TLP3542, J601 RJ45, K601 RELAY_1C, K602 RELAY_1C, M601 W28-XQ1A-10, P601 BATT-IN, P602 CONN_01x02, P603 UMBILICAL, P604 43025-0200, P605 43045-0200, P606 S4B-PH-K, P607 43045-0200, P608 43025-0200, P609 PHR-4, Q601 PMV45EN, Q602 PMV45EN, Q603 ZVN4525E6, Q604 ZVN4525E6, Q605 ZVN4525E6, SW601 SPST, U601 CD74HC14, U602 SN65220DBV, U603 741G08

Commit message: Finished footprint assignment.
Parts:
- D603, D605: footprint Capacitors_ThroughHole:C_Radial_D10_L20_P2.5 -> Choke_Axial_ThroughHole:Choke_Horizontal_RM10mm
- P601, P608: footprint (none) -> Connectors_Molex:Molex_Microfit3_Header_02x01_Straight_43045-0228
- P603: footprint (none) -> Connectors_Molex:Molex_Microfit3_Header_02x05_Straight_43045-1028
Changed lines of the file:
@@
 F 0 "P601" V 15850 950 50  0000 C CNN
 F 1 "BATT-IN" V 15950 950 50  0000 C CNN
-F 2 "" H 15750 950 60  0001 C CNN
+F 2 "Connectors_Molex:Molex_Microfit3_Header_02x01_Straight_43045-0228" H 15750 950 60  0001 C CNN
 F 3 "" H 15750 950 60  0000 C CNN
 	1    15750 950
@@
 F 0 "P603" H 1250 7950 50  0000 C CNN
 F 1 "UMBILICAL" V 1350 7400 50  0000 C CNN
-F 2 "" H 1250 7400 60  0001 C CNN
+F 2 "Connectors_Molex:Molex_Microfit3_Header_02x05_Straight_43045-1028" H 1250 7400 60  0001 C CNN
 F 3 "" H 1250 7400 60  0000 C CNN
 	1    1250 7400
@@
 F 0 "P608" H 14750 8000 50  0000 R CNN
 F 1 "43025-0200" V 14950 7800 50  0000 C CNN
-F 2 "" H 14750 7800 50  0001 C CNN
+F 2 "Connectors_Molex:Molex_Microfit3_Header_02x01_Straight_43045-0228" H 14750 7800 50  0001 C CNN
 F 3 "" H 14750 7800 50  0000 C CNN
 F 4 "MicroFit3 1x2 recept." V 14850 7800 50  0000 C CIN "Note"
@@
 F 0 "D603" V 14599 4142 50  0000 R CNN
 F 1 "LED" V 14508 4142 50  0000 R CNN
-F 2 "Capacitors_ThroughHole:C_Radial_D10_L20_P2.5" H 14500 4250 50  0001 C CNN
+F 2 "Choke_Axial_ThroughHole:Choke_Horizontal_RM10mm" H 14500 4250 50  0001 C CNN
 F 3 "" H 14500 4250 50  0000 C CNN
 F 4 "Ready-To-Launch" V 14409 4142 60  0000 R CIN "Note"
@@
 F 0 "D605" V 9850 7450 50  0000 R CNN
 F 1 "LED" V 9758 7392 50  0001 R CNN
-F 2 "Capacitors_ThroughHole:C_Radial_D10_L20_P2.5" H 9750 7500 50  0001 C CNN
+F 2 "Choke_Axial_ThroughHole:Choke_Horizontal_RM10mm" H 9750 7500 50  0001 C CNN
 F 3 "" H 9750 7500 50  0000 C CNN
 F 4 "Rocket_Ignite" H 9800 7650 60  0000 C CIN "Note"
