File: ltc3/kicad/Launch_Tower_Computer_III.kicad_pcb (KiCad board)
At the start: 2 copper layers, 2 parts

Commit message: More tidying of ltc3/kicad/ tree.
Parts:
- removed BQ77PL900: VAL**, BQ77PL900
- removed LT8490: VAL**, LT8490

Commit message: Updated BQ77PL900 Footprint
Parts:
- added BQ77PL900: VAL**, LTC3:BQ77PL900, F.Cu at (162.6, 113.0)
- added REF**: SSOP-48_7.5x15.9mm_Pitch0.635mm, Housings_SSOP:SSOP-48_7.5x15.9mm_Pitch0.635mm, F.Cu at (162.6, 130.8)

Commit message: LTC3: Cosmetic changes; reference designator updates; etc.
1. Renamed "PHNTM*" reference designators to something more
   conventional and descriptive (e.g., "PHNTM*" to "BT*" for off-board
   batteries).
2. Cosmetic changes to battery management and BeagleBone schematics
   (normalizing text notes style, etc.).
3. Incremental progress on footprint assignment.
4. Imported netlist into PCB layout editor, just for grins.
   Everything fits into a 250x135mm board.  Only $260 for an OSH Park run!
   There may be some opportunities for improvement...
Parts:
- removed BQ77PL900: VAL**, LTC3:BQ77PL900
- removed REF**: SSOP-48_7.5x15.9mm_Pitch0.635mm, Housings_SSOP:SSOP-48_7.5x15.9mm_Pitch0.635mm
- added BT1: ~, Oddities:Dummy_Empty, F.Cu at (262.9, 118.2)
- added BT2: ~, Oddities:Dummy_Empty, F.Cu at (266.3, 121.7)
- added BT3: ~, Oddities:Dummy_Empty, F.Cu at (262.9, 122.8)
- added BT4: ~, Oddities:Dummy_Empty, F.Cu at (259.3, 124.5)
- added BT5: ~, Oddities:Dummy_Empty, F.Cu at (266.5, 117.0)
- added BT6: ~, Oddities:Dummy_Empty, F.Cu at (212.6, 132.6)
- added BT7: ~, Oddities:Dummy_Empty, F.Cu at (253.9, 129.7)
- added BT8: ~, Oddities:Dummy_Empty, F.Cu at (250.5, 130.9)
- added C1: C, Capacitors_SMD:C_0805, F.Cu at (303.1, 155.6)
- added C2: C, Capacitors_SMD:C_0805, F.Cu at (263.0, 162.9)
- added C201: 470n, Capacitors_SMD:C_0805, F.Cu at (131.3, 188.0)
- added C202: 470n, Capacitors_SMD:C_0805, F.Cu at (126.2, 181.6)
- added C203: 33µ, Capacitors_SMD:C_1206, F.Cu at (107.2, 184.4)
- added C204: 33µ, Capacitors_SMD:C_1206, F.Cu at (112.3, 177.6)
- added C205: 33µ, Capacitors_SMD:C_1206, F.Cu at (107.2, 177.6)
- added C206: 2.2µ, Capacitors_SMD:C_0805, F.Cu at (125.2, 162.6)
- added C207: 2.2µ, Capacitors_SMD:C_0805, F.Cu at (139.1, 167.6)
- added C208: 2.2µ, Capacitors_SMD:C_0805, F.Cu at (158.3, 147.3)
- added C209: 2.2µ, Capacitors_SMD:C_0805, F.Cu at (130.7, 175.3)
- added C210: 2.2µ, Capacitors_SMD:C_0805, F.Cu at (130.1, 168.9)
- added C211: 4.7µ, Capacitors_SMD:C_0805, F.Cu at (134.6, 168.0)
- added C212: 4.7µ, Capacitors_SMD:C_0805, F.Cu at (147.0, 153.6)
- added C213: 1μ, Capacitors_SMD:C_0805, F.Cu at (138.8, 161.3)
- added C214: 100n, Capacitors_SMD:C_0805, F.Cu at (112.0, 190.5)
- added C215: 10μ, Capacitors_SMD:C_0805, F.Cu at (153.8, 147.3)
- added C216: 10μ, Capacitors_SMD:C_0805, F.Cu at (126.2, 175.3)
- added C217: 150μ, Capacitors_SMD:C_1206, F.Cu at (133.1, 155.1)
- added C218: 2.2µ, Capacitors_SMD:C_0805, F.Cu at (121.7, 181.6)
- added C219: 0.1μ, Capacitors_SMD:C_0805, F.Cu at (116.5, 188.0)
- added C220: 4.7u, Capacitors_SMD:C_0805, F.Cu at (117.2, 181.7)
- added C221: 1n, Capacitors_SMD:C_0805, F.Cu at (151.5, 153.6)
- added C222: 4.7u, Capacitors_SMD:C_0805, F.Cu at (147.8, 160.0)
- added C223: 220n, Capacitors_SMD:C_0805, F.Cu at (134.3, 161.7)
- added C224: 220n, Capacitors_SMD:C_0805, F.Cu at (149.3, 147.3)
- added C225: 1n, Capacitors_SMD:C_0805, F.Cu at (112.0, 184.2)
- added C226: .18µ, Capacitors_SMD:C_0805, F.Cu at (125.6, 168.9)
- added C227: 1µ, Capacitors_SMD:C_0805, F.Cu at (121.1, 168.9)
- added C228: 100n, Capacitors_SMD:C_0805, F.Cu at (144.8, 147.3)
- added C229: 4.7µ, Capacitors_SMD:C_0805, F.Cu at (140.3, 147.3)
- added C230: 100n, Capacitors_SMD:C_0805, F.Cu at (129.8, 162.6)
- added C231: 10n, Capacitors_SMD:C_0805, F.Cu at (169.5, 153.6)
- added C232: .33µ, Capacitors_SMD:C_0805, F.Cu at (137.9, 154.9)
- added C233: 10n, Capacitors_SMD:C_0805, F.Cu at (117.2, 175.3)
- added C234: 8.2n, Capacitors_SMD:C_0805, F.Cu at (121.7, 175.3)
- added C235: 220p, Capacitors_SMD:C_0805, F.Cu at (142.5, 153.6)
- added C236: 68n, Capacitors_SMD:C_0805, F.Cu at (143.3, 160.0)
- added C3: C, Capacitors_SMD:C_0805, F.Cu at (201.8, 178.3)
- added C301: 0.1μ, Capacitors_SMD:C_0805, F.Cu at (242.9, 103.9)
- added C302: 470p, Capacitors_SMD:C_0805, F.Cu at (249.1, 98.7)
- added C303: 4.7n, Capacitors_SMD:C_0805, F.Cu at (234.2, 115.8)
- added C304: 4.7n, Capacitors_SMD:C_0805, F.Cu at (240.0, 110.3)
- added C305: 2.2μ, Capacitors_SMD:C_0805, F.Cu at (265.4, 105.1)
- added C306: 2.2μ, Capacitors_SMD:C_0805, F.Cu at (241.3, 130.5)
- added C307: 4.7μ, Capacitors_SMD:C_0805, F.Cu at (262.6, 111.4)
- added C308: 1μ, Capacitors_SMD:C_0805, F.Cu at (250.1, 124.1)
- added C309: 1μ, Capacitors_SMD:C_0805, F.Cu at (244.5, 111.4)
- added C310: 0.1μ, Capacitors_SMD:C_0805, F.Cu at (241.0, 117.8)
- added C311: 0.1μ, Capacitors_SMD:C_0805, F.Cu at (245.5, 117.8)
- added C312: 0.1μ, Capacitors_SMD:C_0805, F.Cu at (241.0, 124.1)
- added C313: 2.2μ, Capacitors_SMD:C_0805, F.Cu at (260.9, 105.1)
- added C314: 2.2μ, Capacitors_SMD:C_0805, F.Cu at (267.2, 98.7)
- added C315: 0.1μ, Capacitors_SMD:C_0805, F.Cu at (253.6, 111.4)
- added C316: 10n, Capacitors_SMD:C_0805, F.Cu at (250.1, 117.8)
- added C317: 0.1μ, Capacitors_SMD:C_0805, F.Cu at (245.5, 124.1)
- added C318: 0.1μ, Capacitors_SMD:C_0805, F.Cu at (232.3, 128.5)
- added C319: 0.1μ, Capacitors_SMD:C_0805, F.Cu at (236.8, 130.5)
- added C320: 0.1μ, Capacitors_SMD:C_0805, F.Cu at (259.1, 117.8)
- added C4: C, Capacitors_SMD:C_0805, F.Cu at (234.9, 175.4)
- added C401: 0.1μ, Capacitors_SMD:C_0805, F.Cu at (311.5, 92.4)
- added C402: 1μ, Capacitors_SMD:C_0805, F.Cu at (280.7, 112.8)
- added C403: 2μ2, Capacitors_SMD:C_0805, F.Cu at (298.0, 92.4)
- added C404: 330μ, Capacitors_SMD:C_0805, F.Cu at (291.1, 100.3)
- added C405: 1μ, Capacitors_SMD:C_0805, F.Cu at (285.9, 108.2)
- added C406: 330μ, Capacitors_SMD:C_0805, F.Cu at (286.5, 100.3)
- added C407: 1μ, Capacitors_SMD:C_0805, F.Cu at (309.1, 98.7)
- added C408: 4μ7, Capacitors_SMD:C_0805, F.Cu at (293.5, 92.4)
- added C409: 4μ7, Capacitors_SMD:C_0805, F.Cu at (303.2, 111.4)
- added C410: 4μ7, Capacitors_SMD:C_0805, F.Cu at (304.6, 98.7)
- added C411: 4μ7, Capacitors_SMD:C_0805, F.Cu at (313.6, 98.7)
- added C412: 330μ, Capacitors_SMD:C_0805, F.Cu at (320.6, 92.4)
- added C413: 1μ, Capacitors_SMD:C_0805, F.Cu at (307.7, 105.1)
- added C414: 4μ7, Capacitors_SMD:C_0805, F.Cu at (307.7, 111.4)
- added C415: 4μ7, Capacitors_SMD:C_0805, F.Cu at (303.2, 105.1)
- added C416: 4μ7, Capacitors_SMD:C_0805, F.Cu at (285.2, 114.5)
- added C417: 4μ7, Capacitors_SMD:C_0805, F.Cu at (307.0, 92.4)
- added C501: 0.1μ, Capacitors_SMD:C_0805, F.Cu at (105.6, 207.4)
- added C601: 10μ, Capacitors_SMD:C_1206, F.Cu at (295.4, 155.8)
- added C603: 0.1μ, Capacitors_SMD:C_0805, F.Cu at (318.9, 141.2)
- added C604: 0.1μ, Capacitors_SMD:C_0805, F.Cu at (314.4, 141.2)
- added C605: 0.1μ, Capacitors_SMD:C_0805, F.Cu at (289.8, 165.9)
- added IC1: TLP3542, Housings_DIP:DIP-6_W7.62mm, F.Cu at (280.4, 144.3)
- added IC2: TLP3542, Housings_DIP:DIP-6_W7.62mm, F.Cu at (210.1, 176.3)
- added IC3: TLP3542, Housings_DIP:DIP-6_W7.62mm, F.Cu at (230.7, 164.4)
- added IC4: TLP3542, Housings_DIP:DIP-6_W7.62mm, F.Cu at (243.1, 150.4)
- added IC5: TLP3542, Housings_DIP:DIP-6_W7.62mm, F.Cu at (151.5, 95.5)
- added IC6: TLP3542, Housings_DIP:DIP-6_W7.62mm, F.Cu at (97.8, 126.5)
- added IC7: TLP3542, Housings_DIP:DIP-6_W7.62mm, F.Cu at (118.4, 121.4)
- added IC701: TLP3542, Housings_DIP:DIP-6_W7.62mm, F.Cu at (230.7, 150.4)
- added IC8: TLP3542, Housings_DIP:DIP-6_W7.62mm, F.Cu at (139.0, 95.5)
- added JP1: JUMPER3, Pin_Headers:Pin_Header_Straight_1x03, F.Cu at (144.9, 124.8)
- added JP2: JUMPER3, Pin_Headers:Pin_Header_Straight_1x03, F.Cu at (177.5, 95.4)
- added JP3: JUMPER3, Pin_Headers:Pin_Header_Straight_1x03, F.Cu at (166.4, 104.7)
- added JP4: JUMPER3, Pin_Headers:Pin_Header_Straight_1x03, F.Cu at (158.2, 114.1)
- added JP501: WR_ENABLE, Pin_Headers:Pin_Header_Straight_1x02, F.Cu at (98.8, 203.1)
- added JP601: jumper, Pin_Headers:Pin_Header_Straight_1x02, F.Cu at (279.7, 158.2)
- added L201: 10µH, Inductors:Inductor_1212, F.Cu at (126.8, 155.6)
- added M1: W28-XQ1A-1, Oddities:Dummy_Empty, F.Cu at (257.5, 152.3)
- added M2: W28-XQ1A-1, Oddities:Dummy_Empty, F.Cu at (216.1, 187.7)
- added M3: W28-XQ1A-1, Oddities:Dummy_Empty, F.Cu at (257.5, 147.7)
- added M4: W28-XQ1A-1, Oddities:Dummy_Empty, F.Cu at (205.2, 187.7)
- added M5: W28-XQ1A-0.25, Oddities:Dummy_Empty, F.Cu at (167.1, 92.8)
- added M6: W28-XQ1A-0.25, Oddities:Dummy_Empty, F.Cu at (156.0, 106.8)
- added M7: W28-XQ1A-0.25, Oddities:Dummy_Empty, F.Cu at (147.8, 117.5)
- added M8: W28-XQ1A-0.25, Oddities:Dummy_Empty, F.Cu at (167.1, 97.4)
- added P10: CONN_EXT_PWR_1, Pin_Headers:Pin_Header_Straight_1x02, F.Cu at (113.6, 135.4)
- added P11: CONN_EXT_PWR_3, Pin_Headers:Pin_Header_Straight_1x02, F.Cu at (134.2, 121.3)
- added P12: CONN_EXT_PWR_2, Pin_Headers:Pin_Header_Straight_1x02, F.Cu at (142.4, 109.4)
- added P13: CONN_EXT_PWR_4, Pin_Headers:Pin_Header_Straight_1x02, F.Cu at (127.4, 135.4)
- added P14: CONN_01X10, Pin_Headers:Pin_Header_Straight_1x10, F.Cu at (99.4, 95.4)
- added P15: CONN_01X08, Pin_Headers:Pin_Header_Straight_1x08, F.Cu at (120.1, 95.4)
- added P16: CONN_01X10, Pin_Headers:Pin_Header_Straight_1x10, F.Cu at (109.7, 95.4)
- added P17: CONN_01X08, Pin_Headers:Pin_Header_Straight_1x08, F.Cu at (130.4, 95.4)
- added P201: PV_IN, Pin_Headers:Pin_Header_Straight_1x02, F.Cu at (96.7, 162.3)
- added P202: LAB_IN, Pin_Headers:Pin_Header_Straight_1x02, F.Cu at (97.1, 172.9)
- added P203: S2BPHKS, Pin_Headers:Pin_Header_Straight_1x02, F.Cu at (106.0, 150.3)
- added P3: CONN_EXT_PWR_3, Pin_Headers:Pin_Header_Straight_1x02, F.Cu at (192.8, 181.3)
- added P301: CONN_BATT_MAIN, Pin_Headers:Pin_Header_Straight_1x02, F.Cu at (227.3, 108.1)
- added P302: CONN_BATT_SENSE, Pin_Headers:Pin_Header_Straight_1x02, F.Cu at (235.1, 95.4)
- added P303: S2BPHKS, Pin_Headers:Pin_Header_Straight_1x02, F.Cu at (212.5, 124.5)
- added P304: ~, Oddities:Dummy_Empty, F.Cu at (263.2, 127.5)
- added P305: ~, Oddities:Dummy_Empty, F.Cu at (257.9, 129.7)
- added P4: CONN_EXT_PWR_2, Pin_Headers:Pin_Header_Straight_1x02, F.Cu at (246.5, 164.3)
- added P401: ~, Oddities:Dummy_Empty, F.Cu at (280.4, 119.6)
- added P402: CONN_01X04, Pin_Headers:Pin_Header_Straight_1x04, F.Cu at (279.1, 95.4)
- added P5: CONN_EXT_PWR_4, Pin_Headers:Pin_Header_Straight_1x02, F.Cu at (225.9, 178.4)
- added P6: CONN_01X10, Pin_Headers:Pin_Header_Straight_1x10, F.Cu at (191.1, 150.3)
- added P601: BATT-IN, Pin_Headers:Pin_Header_Straight_1x02, F.Cu at (292.7, 144.2)
- added P602: CONN_01x02, Pin_Headers:Pin_Header_Straight_1x02, F.Cu at (287.7, 158.2)
- added P603: UMBILICAL, Pin_Headers:Pin_Header_Straight_1x10, F.Cu at (272.7, 144.2)
- added P7: CONN_01X08, Pin_Headers:Pin_Header_Straight_1x08, F.Cu at (211.7, 150.3)
- added P701: CONN_EXT_PWR_1, Pin_Headers:Pin_Header_Straight_1x02, F.Cu at (246.5, 175.0)
- added P8: CONN_01X10, Pin_Headers:Pin_Header_Straight_1x10, F.Cu at (201.4, 150.3)
- added P9: CONN_01X08, Pin_Headers:Pin_Header_Straight_1x08, F.Cu at (222.0, 150.3)
- added Q1: PMV45EN, TO_SOT_Packages_SMD:SOT-23, F.Cu at (257.2, 156.7)
- added Q2: PMV45EN, TO_SOT_Packages_SMD:SOT-23, F.Cu at (257.2, 163.4)
- added Q201: Q_NMOS_DGS, LTC3:PG-TDSON-8, F.Cu at (115.2, 149.1)
- added Q202: Q_NMOS_DGS, LTC3:PG-TDSON-8, F.Cu at (107.7, 159.8)
- added Q203: Q_NMOS_DGS, LTC3:PG-TDSON-8, F.Cu at (99.7, 182.5)
- added Q204: Q_NMOS_DGS, LTC3:PG-TDSON-8, F.Cu at (118.0, 158.8)
- added Q205: Q_NPN_BCE, TO_SOT_Packages_SMD:SOT-23, F.Cu at (98.9, 190.5)
- added Q206: Q_PMOS_DGS, LTC3:PG-TDSON-8, F.Cu at (105.2, 169.5)
- added Q207: Q_NPN_BCE, TO_SOT_Packages_SMD:SOT-23, F.Cu at (124.8, 147.4)
- added Q3: PMV45EN, TO_SOT_Packages_SMD:SOT-23, F.Cu at (257.2, 170.1)
- added Q301: NDS9407, Power_Integrations:SO-8, F.Cu at (201.7, 131.1)
- added Q302: MMBT3904, TO_SOT_Packages_SMD:SOT-23, F.Cu at (193.7, 130.6)
- added Q303: SUM110P08-11, TO_SOT_Packages_SMD:TO-263-3Lead, F.Cu at (192.3, 121.3)
- added Q304: SUM110P08-11, TO_SOT_Packages_SMD:TO-263-3Lead, F.Cu at (211.5, 95.9)
- added Q305: SUM110P08-11, TO_SOT_Packages_SMD:TO-263-3Lead, F.Cu at (192.3, 108.6)
- added Q306: SUM110P08-11, TO_SOT_Packages_SMD:TO-263-3Lead, F.Cu at (192.3, 95.9)
- added Q4: PMV45EN, TO_SOT_Packages_SMD:SOT-23, F.Cu at (110.4, 123.6)
- added Q5: PMV45EN, TO_SOT_Packages_SMD:SOT-23, F.Cu at (173.9, 105.8)
- added Q6: PMV45EN, TO_SOT_Packages_SMD:SOT-23, F.Cu at (138.0, 135.2)
- added Q601: PMV45EN, TO_SOT_Packages_SMD:SOT-23, F.Cu at (308.4, 146.5)
- added Q602: PMV45EN, TO_SOT_Packages_SMD:SOT-23, F.Cu at (283.8, 170.7)
- added Q7: PMV45EN, TO_SOT_Packages_SMD:SOT-23, F.Cu at (98.0, 137.6)
- added Q701: PMV45EN, TO_SOT_Packages_SMD:SOT-23, F.Cu at (236.5, 182.8)
- added R1: 30m, Resistors_SMD:R_0805, F.Cu at (235.8, 108.3)
- added R11: 10k, Resistors_SMD:R_0805, F.Cu at (262.8, 169.3)
- added R12: 10k, Resistors_SMD:R_0805, F.Cu at (245.9, 182.7)
- added R13: 270, Resistors_SMD:R_0805, F.Cu at (255.3, 176.7)
- added R14: 270, Resistors_SMD:R_0805, F.Cu at (242.2, 182.7)
- added R17: 10k, Resistors_SMD:R_0805, F.Cu at (183.1, 92.4)
- added R18: 10k, Resistors_SMD:R_0805, F.Cu at (154.2, 124.3)
- added R19: 270, Resistors_SMD:R_0805, F.Cu at (150.5, 128.1)
- added R2: 10k, Resistors_SMD:R_0805, F.Cu at (290.0, 106.6)
- added R20: 270, Resistors_SMD:R_0805, F.Cu at (143.7, 135.0)
- added R201: 30m, Resistors_SMD:R_0805, F.Cu at (172.2, 147.3)
- added R202: 10, Resistors_SMD:R_0805, F.Cu at (153.2, 166.3)
- added R203: 10, Resistors_SMD:R_0805, F.Cu at (140.0, 180.3)
- added R204: 5m, Resistors_SMD:R_0805, F.Cu at (161.9, 160.0)
- added R205: 5m, Resistors_SMD:R_0805, F.Cu at (144.5, 179.0)
- added R206: 600, Resistors_SMD:R_0805, F.Cu at (157.7, 166.3)
- added R21: 10k, Resistors_SMD:R_0805, F.Cu at (150.5, 121.8)
- added R211: 0, Resistors_SMD:R_0805, F.Cu at (176.7, 147.3)
- added R212: 10, Resistors_SMD:R_0805, F.Cu at (135.8, 187.1)
- added R213: 5m, Resistors_SMD:R_0805, F.Cu at (145.1, 185.4)
- added R214: 600, Resistors_SMD:R_0805, F.Cu at (167.1, 166.3)
- added R215: 10, Resistors_SMD:R_0805, F.Cu at (162.9, 172.7)
- added R216: 196k, Resistors_SMD:R_0805, F.Cu at (171.6, 166.3)
- added R217: 100k, Resistors_SMD:R_0805, F.Cu at (149.6, 185.4)
- added R218: 8.06k, Resistors_SMD:R_0805, F.Cu at (149.2, 172.7)
- added R219: 33k, Resistors_SMD:R_0805, F.Cu at (158.3, 172.7)
- added R22: 10k, Resistors_SMD:R_0805, F.Cu at (103.6, 137.5)
- added R220: 100k, Resistors_SMD:R_0805, F.Cu at (171.2, 160.0)
- added R221: 294k, Resistors_SMD:R_0805, F.Cu at (178.8, 153.6)
- added R222: 11.5k, Resistors_SMD:R_0805, F.Cu at (144.4, 172.7)
- added R223: 57.6k, Resistors_SMD:R_0805, F.Cu at (153.7, 179.0)
- added R224: 10.2k, Resistors_SMD:R_0805, F.Cu at (162.4, 166.3)
- added R225: 11.5k, Resistors_SMD:R_0805, F.Cu at (140.5, 186.7)
- added R226: 110k, Resistors_SMD:R_0805, F.Cu at (149.0, 179.0)
- added R227: 93.1k, Resistors_SMD:R_0805, F.Cu at (174.2, 153.6)
- added R228: 26.1k, Resistors_SMD:R_0805, F.Cu at (166.6, 160.0)
- added R229: 215k, Resistors_SMD:R_0805, F.Cu at (153.8, 172.7)
- added R23: 270, Resistors_SMD:R_0805, F.Cu at (163.8, 114.9)
- added R230: 35.7k, Resistors_SMD:R_0805, F.Cu at (152.5, 160.0)
- added R231: 7.68k, Resistors_SMD:R_0805, F.Cu at (157.3, 160.0)
- added R232: 16.5k, Resistors_SMD:R_0805, F.Cu at (121.8, 188.0)
- added R233: 21k, Resistors_SMD:R_0805, F.Cu at (165.0, 153.6)
- added R234: 3.32k, Resistors_SMD:R_0805, F.Cu at (126.6, 188.0)
- added R235: 27.1k, Resistors_SMD:R_0805, F.Cu at (167.5, 147.3)
- added R236: 3.01k, Resistors_SMD:R_0805, F.Cu at (148.6, 166.3)
- added R237: 1.3k, Resistors_SMD:R_0805, F.Cu at (160.5, 153.6)
- added R238: 243k, Resistors_SMD:R_0805, F.Cu at (139.7, 174.0)
- added R239: 10k, Resistors_SMD:R_0805, F.Cu at (135.5, 180.7)
- added R24: 270, Resistors_SMD:R_0805, F.Cu at (172.0, 112.3)
- added R240: 53.6k, Resistors_SMD:R_0805, F.Cu at (130.9, 181.6)
- added R241: 3.32k, Resistors_SMD:R_0805, F.Cu at (143.8, 166.3)
- added R242: 549, Resistors_SMD:R_0805, F.Cu at (135.2, 174.4)
- added R243: 549, Resistors_SMD:R_0805, F.Cu at (162.9, 147.3)
- added R244: 200k, Resistors_SMD:R_0805, F.Cu at (156.0, 153.6)
- added R3: 100k, Resistors_SMD:R_0805, F.Cu at (290.3, 113.0)
- added R301: 5k6, Resistors_SMD:R_0805, F.Cu at (223.0, 121.0)
- added R302: 390k, Resistors_SMD:R_0805, F.Cu at (218.5, 121.5)
- added R303: 1.78k, Resistors_SMD:R_0805, F.Cu at (251.5, 92.4)
- added R304: 820k, Resistors_SMD:R_0805, F.Cu at (244.6, 97.6)
- added R305: 10k, Resistors_SMD:R_0805, F.Cu at (256.2, 92.4)
- added R306: 1M, Resistors_SMD:R_0805, F.Cu at (227.5, 122.1)
- added R307: 1M, Resistors_SMD:R_0805, F.Cu at (218.5, 127.8)
- added R308: 100k, Resistors_SMD:R_0805, F.Cu at (223.0, 127.3)
- added R309: 1k, Resistors_SMD:R_0805, F.Cu at (253.6, 98.7)
- added R310: 1k, Resistors_SMD:R_0805, F.Cu at (229.7, 115.8)
- added R311: 500, Resistors_SMD:R_0805, F.Cu at (260.7, 92.4)
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Other:
- board outline added: 250 x 135 mm

Commit message: LTC3: More component values and footprint assignments.
Split the two-in-one Beagle Bone expansion header component into two
separate components.  Otherwise, we'd be stuck with having to use a
single footprint for the BB cape pin headers, which means pin
numbering that doesn't match the BB docs.
Parts:
- removed BT1, BT2, BT3, BT4, BT5, BT6, BT7, BT8: ~, Oddities:Dummy_Empty
- removed C1, C2, C3, C4: C, Capacitors_SMD:C_0805
- removed IC1, IC2, IC3, IC4, IC5, IC6, IC7, IC8: TLP3542, Housings_DIP:DIP-6_W7.62mm
- removed JP1, JP2, JP3, JP4: JUMPER3, Pin_Headers:Pin_Header_Straight_1x03
- removed M1, M2, M3, M4: W28-XQ1A-1, Oddities:Dummy_Empty
- removed M5, M6, M7, M8: W28-XQ1A-0.25, Oddities:Dummy_Empty
- removed P10: CONN_EXT_PWR_1, Pin_Headers:Pin_Header_Straight_1x02
- removed P11, P3: CONN_EXT_PWR_3, Pin_Headers:Pin_Header_Straight_1x02
- removed P12, P4: CONN_EXT_PWR_2, Pin_Headers:Pin_Header_Straight_1x02
- removed P13, P5: CONN_EXT_PWR_4, Pin_Headers:Pin_Header_Straight_1x02
- removed P14, P16, P6, P8: CONN_01X10, Pin_Headers:Pin_Header_Straight_1x10
- removed P15, P17, P7, P9: CONN_01X08, Pin_Headers:Pin_Header_Straight_1x08
- removed Q1, Q2, Q3, Q4, Q5, Q6, Q7: PMV45EN, TO_SOT_Packages_SMD:SOT-23
- removed R1: 30m, Resistors_SMD:R_0805
- removed R11, R12, R17, R18, R2, R21, R22, R6, R8: 10k, Resistors_SMD:R_0805
- removed R13, R14, R19, R20, R23, R24, R9: 270, Resistors_SMD:R_0805
- removed R243: 549, Resistors_SMD:R_0805
- removed R244: 200k, Resistors_SMD:R_0805
- removed R3, R7: 100k, Resistors_SMD:R_0805
- removed SW1, SW10, SW11, SW2, SW4, SW5, SW6, SW7, SW8, SW9: SP3T, Oddities:Dummy_Empty
- removed SW3: SPST_switch, Oddities:Dummy_Empty
- removed U604: 741G08, TO_SOT_Packages_SMD:SOT-353
- removed W1, W10, W11, W12, W13, W14, W15, W16, W17, W18, W19, W2, W28, W29, W3, W4, W5, W6, W7, W8, W9: TEST, Measurement_Points:Test_Point_2Pads
- removed W20, W21, W22, W23, W25: 0/5V, Measurement_Points:Test_Point_2Pads
- removed W24: 0/3.3V, Measurement_Points:Test_Point_2Pads
- removed W26: 14.8-16.8V, Measurement_Points:Test_Point_2Pads
- removed W27: 0/14.8-16.8V, Measurement_Points:Test_Point_2Pads
- removed W30, W31, W32: TEST_1P, Measurement_Points:Test_Point_2Pads
- added BT301: ~, Oddities:Dummy_Empty, F.Cu at (532.8, 175.1)
- added BT302: ~, Oddities:Dummy_Empty, F.Cu at (565.0, 144.5)
- added BT303: ~, Oddities:Dummy_Empty, F.Cu at (535.1, 170.4)
- added BT304: ~, Oddities:Dummy_Empty, F.Cu at (565.0, 139.9)
- added BT305: ~, Oddities:Dummy_Empty, F.Cu at (548.4, 159.2)
- added BT306: ~, Oddities:Dummy_Empty, F.Cu at (558.6, 148.9)
- added BT307: ~, Oddities:Dummy_Empty, F.Cu at (575.5, 132.3)
- added BT308: ~, Oddities:Dummy_Empty, F.Cu at (495.1, 175.2)
- added C606: 0.1μ, Capacitors_SMD:C_0805, F.Cu at (793.1, 112.4)
- added C702: 1μ, Capacitors_SMD:C_0805, F.Cu at (685.3, 133.6)
- added C703: 1μ, Capacitors_SMD:C_0805, F.Cu at (653.5, 163.7)
- added C704: 1μ, Capacitors_SMD:C_0805, F.Cu at (673.3, 140.3)
- added D301: 1SS355, Diodes_SMD:TUMD2, F.Cu at (489.3, 174.6)
- added D302: SMAZ16, Diodes_SMD:SMA_Standard, F.Cu at (551.2, 124.8)
- added D303: SMAZ16, Diodes_SMD:SMA_Standard, F.Cu at (531.3, 140.0)
- added D304: 1SS355, Diodes_SMD:TUMD2, F.Cu at (482.9, 174.6)
- added D305: SMAZ16, Diodes_SMD:SMA_Standard, F.Cu at (551.2, 114.6)
- added D306: SMAZ16, Diodes_SMD:SMA_Standard, F.Cu at (558.7, 114.6)
- added D601: CDSU4148, Resistors_SMD:R_0603, F.Cu at (761.4, 124.1)
- added D602: CDSU4148, Resistors_SMD:R_0603, F.Cu at (771.5, 119.7)
- added D604: CDSU4148, Resistors_SMD:R_0603, F.Cu at (725.4, 148.8)
- added D609: 3.3V, Diodes_SMD:SMA_Standard, F.Cu at (753.4, 126.1)
- added IC601: TLP3542, Housings_DIP:DIP-6_W7.62mm, F.Cu at (770.8, 102.8)
- added IC702: TLP3542, Housings_DIP:DIP-6_W7.62mm, F.Cu at (677.5, 116.0)
- added IC703: TLP3542, Housings_DIP:DIP-6_W7.62mm, F.Cu at (599.6, 165.3)
- added IC704: TLP3542, Housings_DIP:DIP-6_W7.62mm, F.Cu at (587.1, 165.3)
- added IC801: TLP3542, Housings_DIP:DIP-6_W7.62mm, F.Cu at (578.5, 33.2)
- added IC802: TLP3542, Housings_DIP:DIP-6_W7.62mm, F.Cu at (566.1, 47.3)
- added IC803: TLP3542, Housings_DIP:DIP-6_W7.62mm, F.Cu at (531.3, 82.5)
- added IC804: TLP3542, Housings_DIP:DIP-6_W7.62mm, F.Cu at (566.1, 33.2)
- added J601: RJ45, Connect:RJ45_8, F.Cu at (741.6, 131.7)
- added JP801: Trigger Level, Pin_Headers:Pin_Header_Straight_1x03, F.Cu at (533.0, 96.4)
- added JP802: Trigger Level, Pin_Headers:Pin_Header_Straight_1x03, F.Cu at (580.2, 47.2)
- added JP803: Trigger Level, Pin_Headers:Pin_Header_Straight_1x03, F.Cu at (566.6, 61.2)
- added JP804: Trigger Level, Pin_Headers:Pin_Header_Straight_1x03, F.Cu at (592.6, 33.1)
- added M701: W28-XQ1A-1, Oddities:Dummy_Empty, F.Cu at (626.4, 167.2)
- added M702: W28-XQ1A-1, Oddities:Dummy_Empty, F.Cu at (637.4, 162.5)
- added M703: W28-XQ1A-1, Oddities:Dummy_Empty, F.Cu at (658.5, 152.8)
- added M704: W28-XQ1A-1, Oddities:Dummy_Empty, F.Cu at (626.4, 162.5)
- added M801: W28-XQ1A-0.25, Oddities:Dummy_Empty, F.Cu at (466.2, 104.4)
- added M802: W28-XQ1A-0.25, Oddities:Dummy_Empty, F.Cu at (506.1, 104.4)
- added M803: W28-XQ1A-0.25, Oddities:Dummy_Empty, F.Cu at (492.8, 104.4)
- added M804: W28-XQ1A-0.25, Oddities:Dummy_Empty, F.Cu at (479.5, 104.4)
- added P306: CONN_01X02, Valves:VALVE-OCTAL, F.Cu at (506.9, 122.1)
- added P501: BeagleBone_Black_Expansion_Header_P8, Pin_Headers:Pin_Header_Straight_2x23, B.Cu at (203.9, 76.2)
- added P502: BeagleBone_Black_Expansion_Header_P9, Pin_Headers:Pin_Header_Straight_2x23, B.Cu at (252.2, 76.2)
- added P702: CONN_01X10, Oddities:Dummy_Empty, F.Cu at (691.6, 113.3)
- added P703: CONN_EXT_PWR_1, Valves:VALVE-OCTAL, F.Cu at (630.7, 122.1)
- added P704: CONN_EXT_PWR_2, Valves:VALVE-OCTAL, F.Cu at (595.9, 146.7)
- added P705: CONN_01X08, Connectors_Molex:Molex_Microfit3_Header_02x04_Angled_43045-080x, F.Cu at (666.5, 137.1)
- added P706: CONN_01X08, Oddities:Dummy_Empty, F.Cu at (637.1, 167.2)
- added P707: CONN_EXT_PWR_3, Valves:VALVE-OCTAL, F.Cu at (595.9, 122.1)
- added P708: CONN_EXT_PWR_4, Valves:VALVE-OCTAL, F.Cu at (630.7, 146.7)
- added P801: CONN_01X10, Valves:VALVE-OCTAL, F.Cu at (506.5, 63.9)
- added P802: CONN_01X10, Valves:VALVE-OCTAL, F.Cu at (540.1, 63.9)
- added P803: CONN_EXT_PWR_1, Valves:VALVE-OCTAL, F.Cu at (471.8, 39.3)
- added P804: CONN_EXT_PWR_2, Valves:VALVE-OCTAL, F.Cu at (471.8, 63.9)
- added P805: CONN_01X08, Valves:VALVE-OCTAL, F.Cu at (541.2, 39.3)
- added P806: CONN_01X08, Valves:VALVE-OCTAL, F.Cu at (506.5, 88.6)
- added P807: CONN_EXT_PWR_3, Valves:VALVE-OCTAL, F.Cu at (506.5, 39.3)
- added P808: CONN_EXT_PWR_4, Valves:VALVE-OCTAL, F.Cu at (471.8, 88.6)
- added Q702: PMV45EN, TO_SOT_Packages_SMD:SOT-23, F.Cu at (674.8, 133.8)
- added Q703: PMV45EN, TO_SOT_Packages_SMD:SOT-23, F.Cu at (656.8, 157.2)
- added Q704: PMV45EN, TO_SOT_Packages_SMD:SOT-23, F.Cu at (685.3, 127.1)
- added Q801: PMV45EN, TO_SOT_Packages_SMD:SOT-23, F.Cu at (544.0, 79.5)
- added Q802: PMV45EN, TO_SOT_Packages_SMD:SOT-23, F.Cu at (551.5, 79.5)
- added Q803: PMV45EN, TO_SOT_Packages_SMD:SOT-23, F.Cu at (544.0, 86.2)
- added Q804: PMV45EN, TO_SOT_Packages_SMD:SOT-23, F.Cu at (551.5, 86.2)
- added R209: 0, Resistors_SMD:R_0805, F.Cu at (678.0, 60.5)
- added R210: 10, Resistors_SMD:R_0805, F.Cu at (712.8, 36.5)
- added R324: 1m, Resistors_SMD:R_0805, F.Cu at (572.2, 112.9)
- added R409: 10k, Resistors_SMD:R_0805, F.Cu at (759.2, 62.2)
- added R410: 2k91, Resistors_SMD:R_0805, F.Cu at (777.1, 30.1)
- added R619: 10k, Resistors_SMD:R_0805, F.Cu at (788.6, 118.8)
- added R620: 10k, Resistors_SMD:R_0805, F.Cu at (767.9, 125.9)
- added R622: 10k, Resistors_SMD:R_0805, F.Cu at (767.0, 132.2)
- added R702: 270, Resistors_SMD:R_0805, F.Cu at (677.8, 140.3)
- added R705: 10k, Resistors_SMD:R_0805, F.Cu at (644.5, 166.8)
- added R706: 10k, Resistors_SMD:R_0805, F.Cu at (680.8, 133.6)
- added R707: 270, Resistors_SMD:R_0805, F.Cu at (649.0, 168.5)
- added R708: 270, Resistors_SMD:R_0805, F.Cu at (649.0, 162.1)
- added R711: 10k, Resistors_SMD:R_0805, F.Cu at (691.3, 123.9)
- added R712: 10k, Resistors_SMD:R_0805, F.Cu at (666.2, 152.4)
- added R801: 270, Resistors_SMD:R_0805, F.Cu at (542.5, 92.8)
- added R802: 270, Resistors_SMD:R_0805, F.Cu at (589.7, 43.4)
- added R803: 10k, Resistors_SMD:R_0805, F.Cu at (583.1, 57.4)
- added R804: 10k, Resistors_SMD:R_0805, F.Cu at (547.0, 92.8)
- added R805: 270, Resistors_SMD:R_0805, F.Cu at (578.6, 57.4)
- added R806: 270, Resistors_SMD:R_0805, F.Cu at (557.5, 79.4)
- added R807: 10k, Resistors_SMD:R_0805, F.Cu at (563.7, 71.5)
- added R808: 10k, Resistors_SMD:R_0805, F.Cu at (574.1, 58.2)
- added REF**: BeagleBone_Outline, LTC3:BeagleBone_Outline, F.Cu at (202.7, 76.2)
- added SW401: SPST_switch, Oddities:Dummy_Empty, F.Cu at (764.1, 45.3)
- added SW402: SP3T, Oddities:Dummy_Empty, F.Cu at (795.7, 36.7)
- added SW403: SP3T, Oddities:Dummy_Empty, F.Cu at (780.7, 55.7)
- added SW701: SP3T, Oddities:Dummy_Empty, F.Cu at (634.9, 171.8)
- added SW702: SP3T, Oddities:Dummy_Empty, F.Cu at (663.3, 159.1)
- added SW703: SP3T, Oddities:Dummy_Empty, F.Cu at (629.3, 171.8)
- added SW704: SP3T, Oddities:Dummy_Empty, F.Cu at (623.7, 171.8)
- added SW801: SP3T, Oddities:Dummy_Empty, F.Cu at (562.5, 79.8)
- added SW802: SP3T, Oddities:Dummy_Empty, F.Cu at (579.1, 64.2)
- added SW803: SP3T, Oddities:Dummy_Empty, F.Cu at (521.1, 104.4)
- added SW804: SP3T, Oddities:Dummy_Empty, F.Cu at (515.5, 104.4)
- added U601: CD74HC14, Housings_SSOP:TSSOP-14_4.4x5mm_Pitch0.65mm, F.Cu at (783.9, 101.2)
- added W201: TEST, Measurement_Points:Test_Point_2Pads, F.Cu at (712.5, 42.7)
- added W202: TEST, Measurement_Points:Test_Point_2Pads, F.Cu at (688.9, 75.8)
- added W203: TEST, Measurement_Points:Test_Point_2Pads, F.Cu at (712.5, 48.9)
- added W204: TEST, Measurement_Points:Test_Point_2Pads, F.Cu at (718.1, 42.7)
- added W205: TEST, Measurement_Points:Test_Point_2Pads, F.Cu at (701.0, 61.8)
- added W206: TEST, Measurement_Points:Test_Point_2Pads, F.Cu at (690.1, 69.4)
- added W207: TEST, Measurement_Points:Test_Point_2Pads, F.Cu at (673.7, 86.8)
- added W208: TEST, Measurement_Points:Test_Point_2Pads, F.Cu at (683.3, 75.8)
- added W209: TEST, Measurement_Points:Test_Point_2Pads, F.Cu at (695.4, 61.8)
- added W210: TEST, Measurement_Points:Test_Point_2Pads, F.Cu at (703.4, 55.4)
- added W301: TEST, Measurement_Points:Test_Point_2Pads, F.Cu at (520.5, 174.7)
- added W302: TEST, Measurement_Points:Test_Point_2Pads, F.Cu at (526.2, 174.7)
- added W303: TEST, Measurement_Points:Test_Point_2Pads, F.Cu at (552.0, 148.4)
- added W304: TEST_1P, Measurement_Points:Test_Point_2Pads, F.Cu at (461.6, 174.7)
- added W305: TEST_1P, Measurement_Points:Test_Point_2Pads, F.Cu at (468.4, 174.7)
- added W306: TEST_1P, Measurement_Points:Test_Point_2Pads, F.Cu at (475.1, 174.7)
- added W401: TEST, Measurement_Points:Test_Point_2Pads, F.Cu at (779.6, 49.1)
- added W402: TEST, Measurement_Points:Test_Point_2Pads, F.Cu at (770.0, 57.5)
- added W403: TEST, Measurement_Points:Test_Point_2Pads, F.Cu at (763.0, 63.8)
- added W404: TEST, Measurement_Points:Test_Point_2Pads, F.Cu at (768.7, 63.8)
- added W405: TEST, Measurement_Points:Test_Point_2Pads, F.Cu at (788.6, 42.7)
- added W406: TEST, Measurement_Points:Test_Point_2Pads, F.Cu at (794.5, 30.0)
- added W501: TEST, Measurement_Points:Test_Point_2Pads, F.Cu at (258.5, 97.0)
- added W502: TEST, Measurement_Points:Test_Point_2Pads, F.Cu at (258.5, 101.0)
- added W601: 14.8-16.8V, Measurement_Points:Test_Point_2Pads, F.Cu at (770.7, 113.7)
- added W602: 0/5V, Measurement_Points:Test_Point_2Pads, F.Cu at (779.9, 134.1)
- added W603: 0/5V, Measurement_Points:Test_Point_2Pads, F.Cu at (792.4, 118.7)
- added W604: 0/5V, Measurement_Points:Test_Point_2Pads, F.Cu at (780.8, 127.9)
- added W605: 0/5V, Measurement_Points:Test_Point_2Pads, F.Cu at (786.4, 125.0)
- added W606: 0/5V, Measurement_Points:Test_Point_2Pads, F.Cu at (766.4, 144.8)
- added W607: 0/3.3V, Measurement_Points:Test_Point_2Pads, F.Cu at (772.2, 139.5)
- added W608: 0/14.8-16.8V, Measurement_Points:Test_Point_2Pads, F.Cu at (704.4, 148.9)
- C217: footprint Capacitors_SMD:C_1206 -> Capacitors_ThroughHole:C_Radial_D12.5_L25_P5
- C404, C406, C412: value 330μ -> 470μ; footprint Capacitors_SMD:C_0805 -> Capacitors_ThroughHole:C_Radial_D10_L25_P5
- C604: value 0.1μ -> 1μ
- JP601: value jumper -> Shorting Bar
- P201, P202, P203, P301, P601, P602: footprint Pin_Headers:Pin_Header_Straight_1x02 -> Valves:VALVE-OCTAL
- P302: value CONN_BATT_SENSE -> ~; footprint Pin_Headers:Pin_Header_Straight_1x02 -> Oddities:Dummy_Empty
- P303: value S2BPHKS -> CONN_BATT_SENSE; footprint Pin_Headers:Pin_Header_Straight_1x02 -> Valves:VALVE-OCTAL
- P305: value ~ -> S2BPHKS; footprint Oddities:Dummy_Empty -> Valves:VALVE-OCTAL
- P402: footprint Pin_Headers:Pin_Header_Straight_1x04 -> Valves:VALVE-OCTAL
- P603: footprint Pin_Headers:Pin_Header_Straight_1x10 -> Valves:VALVE-OCTAL
- P701: value CONN_EXT_PWR_1 -> CONN_01X10; footprint Pin_Headers:Pin_Header_Straight_1x02 -> Connectors_Molex:Molex_Microfit3_Header_02x05_Angled_43045-100x
- Q201, Q202, Q203, Q204: value Q_NMOS_DGS -> BSC028N06NS
- Q205: value Q_NPN_BCE -> ZVN4525E6
- Q301: value NDS9407 -> MMBT3904; footprint Power_Integrations:SO-8 -> TO_SOT_Packages_SMD:SOT-23
- Q302: value MMBT3904 -> SUM110P08-11; footprint TO_SOT_Packages_SMD:SOT-23 -> TO_SOT_Packages_SMD:TO-263-3Lead
- Q306: value SUM110P08-11 -> NDS9407; footprint TO_SOT_Packages_SMD:TO-263-3Lead -> Power_Integrations:SO-8
- R201: value 30m -> 10
- R203: value 10 -> 5m
- R205: value 5m -> 30m
- R211: value 0 -> 5m
- R212: value 10 -> 600
- R213: value 5m -> 10
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Connections:
- C604 pad 1: +5V -> /Rocket Umbilical & Ignition Control/UMB_DISCONN
- P303 pad 1: Net-(C316-Pad1) -> Net-(C310-Pad1)
- P303 pad 2: GND -> Net-(C310-Pad2)
- P603 pad 3: (no net) -> /Rocket Umbilical & Ignition Control/ROCKET_ETH_1
- P603 pad 4: (no net) -> /Rocket Umbilical & Ignition Control/ROCKET_ETH_2
- P603 pad 5: (no net) -> /Rocket Umbilical & Ignition Control/ROCKET_ETH_3
- P603 pad 6: (no net) -> /Rocket Umbilical & Ignition Control/ROCKET_ETH_4
- P603 pad 7: (no net) -> /Rocket Umbilical & Ignition Control/UMB_CONN_FROM_RKT
- P701 pad 1: Net-(C701-Pad1) -> /External Device Power/EXT_POW_1_FET_D
- P701 pad 2: GND -> /External Device Power/EXT_POW_1_LED_CATH
- Q301 pad 1: Net-(C304-Pad1) -> Net-(C302-Pad1)
- Q301 pad 2: Net-(C304-Pad1) -> Net-(C302-Pad1)
- Q301 pad 3: Net-(C304-Pad1) -> Net-(C302-Pad2)
- Q302 pad 1: Net-(C302-Pad1) -> Net-(C303-Pad2)
- Q302 pad 2: Net-(C302-Pad1) -> Net-(Q302-Pad2)
- Q302 pad 3: Net-(C302-Pad2) -> VBATT
- Q303 pad 1: Net-(C303-Pad2) -> Net-(C304-Pad2)
- Q303 pad 2: Net-(Q303-Pad2) -> Net-(Q302-Pad2)
- Q303 pad 3: VBATT -> Net-(C304-Pad1)
- Q304 pad 1: Net-(C304-Pad2) -> Net-(C303-Pad2)
- Q304 pad 2: Net-(Q303-Pad2) -> Net-(Q302-Pad2)
- Q304 pad 3: Net-(C304-Pad1) -> VBATT
- Q305 pad 1: Net-(C303-Pad2) -> Net-(C304-Pad2)
- Q305 pad 2: Net-(Q303-Pad2) -> Net-(Q302-Pad2)
- Q305 pad 3: VBATT -> Net-(C304-Pad1)
- Q306 pad 1: Net-(C304-Pad2) -> Net-(C304-Pad1)
- Q306 pad 2: Net-(Q303-Pad2) -> Net-(C304-Pad1)
- Q306 pad 4: (no net) -> Net-(Q306-Pad4)
- Q601 pad 3: (no net) -> Net-(D601-Pad2)
- Q602 pad 3: (no net) -> Net-(D604-Pad2)
- R201 pad 1: VBATT -> Net-(C209-Pad1)
- R201 pad 2: Net-(C215-Pad1) -> Net-(C201-Pad1)
- R202 pad 1: Net-(C209-Pad1) -> Net-(C215-Pad1)
- R202 pad 2: Net-(C201-Pad1) -> Net-(C202-Pad1)
- R203 pad 1: Net-(C215-Pad1) -> Net-(C209-Pad1)
- R203 pad 2: Net-(C202-Pad1) -> VBATT
- R204 pad 1: Net-(C209-Pad1) -> Net-(C215-Pad1)
- R204 pad 2: VBATT -> /Power In, Battery Charge & PV MPPT/EXTVCC
- R205 pad 1: Net-(C215-Pad1) -> VBATT
- R205 pad 2: /Power In, Battery Charge & PV MPPT/EXTVCC -> Net-(C215-Pad1)
- R211 pad 1: Net-(C220-Pad1) -> Net-(Q203-Pad3)
- R211 pad 2: (no net) -> GND
- R212 pad 1: Net-(C221-Pad1) -> Net-(R212-Pad1)
- R212 pad 2: Net-(Q203-Pad3) -> GND
- R213 pad 1: Net-(Q203-Pad3) -> Net-(C225-Pad1)
- R214 pad 1: Net-(R214-Pad1) -> VBATT
- R214 pad 2: GND -> Net-(Q205-Pad1)
- R215 pad 1: Net-(C225-Pad1) -> Net-(F201-Pad2)
- R215 pad 2: GND -> Net-(Q205-Pad2)
- R216 pad 1: VBATT -> Net-(Q205-Pad1)
- R216 pad 2: Net-(Q205-Pad2) -> GND
- R217 pad 1: Net-(F1-Pad2) -> Net-(Q205-Pad2)
- R217 pad 2: Net-(Q205-Pad1) -> GND
- R218 pad 1: Net-(Q205-Pad2) -> VBATT
- R218 pad 2: GND -> Net-(D203-Pad2)
- R219 pad 1: Net-(Q205-Pad1) -> Net-(Q206-Pad1)
- R219 pad 2: GND -> Net-(R219-Pad2)
- R220 pad 1: VBATT -> Net-(C226-Pad1)
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Routing:
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
Commit message: LTC3: Spec'd parts for external power and trigger schematics.
Assigned part numbers, footprints to switch and breaker connectors.

Also updated netlist, schematic PDF.
Parts:
- added C701: 1μ, Capacitors_SMD:C_0805, F.Cu at (554.1, 205.5)
- added D201: CMMR1U-02, Diodes_SMD:SOD-123, F.Cu at (462.0, 174.8)
- added D202: CMMR1U-02, Diodes_SMD:SOD-123, F.Cu at (482.5, 172.2)
- added F201: 15A, LTC3:Fuseholder_Auto_Blade_Regular_Keystone_3557-2, F.Cu at (467.2, 165.1)
- added F301: 10A, LTC3:Fuseholder_Auto_Blade_Regular_Keystone_3557-2, F.Cu at (467.2, 93.0)
- added F601: FUSE, LTC3:Fuseholder_Auto_Blade_Regular_Keystone_3557-2, F.Cu at (591.8, 165.1)
- added P604: CONN_01x02, Oddities:Dummy_Empty, F.Cu at (607.2, 169.1)
- added P605: CONN_01x02, Valves:VALVE-OCTAL, F.Cu at (627.5, 147.1)
- added R207: 0, Resistors_SMD:R_0805, F.Cu at (528.8, 160.4)
- added R208: 0, Resistors_SMD:R_0805, F.Cu at (533.3, 155.2)
- added R621: 5.1k, Resistors_SMD:R_0805, F.Cu at (689.8, 119.6)
- added R703: 51k, Resistors_SMD:R_0805, F.Cu at (522.5, 240.3)
- added R704: 51k, Resistors_SMD:R_0805, F.Cu at (522.5, 234.0)
- added R710: 51k, Resistors_SMD:R_0805, F.Cu at (539.6, 224.2)
- added W307: TEST_1P, Measurement_Points:Measurement_Point_Round-TH_Small, F.Cu at (476.3, 103.0)
- JP601: footprint Pin_Headers:Pin_Header_Straight_1x02 -> Oddities:Dummy_Empty
- P701: value CONN_01X10 -> 43045-1000
- P702: value CONN_01X10 -> 43025-1000
- P705: value CONN_01X08 -> 43045-0800
- P706: value CONN_01X08 -> 43025-0800
- P801: value CONN_01X10 -> 43045-1000; footprint Valves:VALVE-OCTAL -> Connectors_Molex:Molex_Microfit3_Header_02x05_Angled_43045-100x
- P802: value CONN_01X10 -> 43025-1000; footprint Valves:VALVE-OCTAL -> Oddities:Dummy_Empty
- P805: value CONN_01X08 -> 43045-0800; footprint Valves:VALVE-OCTAL -> Connectors_Molex:Molex_Microfit3_Header_02x04_Angled_43045-080x
- P806: value CONN_01X08 -> 43025-0800; footprint Valves:VALVE-OCTAL -> Oddities:Dummy_Empty
- Q205: footprint TO_SOT_Packages_SMD:SOT-23 -> LTC3:SOT-26
- W304, W305, W306: footprint Measurement_Points:Test_Point_2Pads -> Measurement_Points:Measurement_Point_Round-SMD-Pad_Small
- moved R213 243.4 mm to (500.3, 171.3)
- moved C213 240.4 mm to (514.2, 166.7)
- moved C229 240.3 mm to (523.5, 173.1)
- moved R241 223.3 mm to (504.8, 168.4)
- moved Q205 221.5 mm to (493.5, 165.3)
- moved C214 221.0 mm to (509.4, 155.3)
- moved P702 220.5 mm to (510.5, 239.0)
- moved R230 218.3 mm to (528.5, 166.8)
- moved C220 214.6 mm to (526.7, 135.0)
- moved R215 214.4 mm to (495.0, 171.8)
- moved W210 211.7 mm to (527.4, 173.0)
- moved C202 211.3 mm to (504.8, 162.0)
- moved P203 210.5 mm to (469.3, 147.1)
- moved C203 210.3 mm to (490.1, 172.5)
- moved C207 209.8 mm to (504.8, 174.7)
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Connections:
- P202 pad 2: (no net) -> Net-(F201-Pad1)
- P301 pad 1: (no net) -> Net-(F301-Pad2)
- P306 pad 1: (no net) -> Net-(P306-Pad1)
- P602 pad 1: Net-(JP601-Pad1) -> Net-(P602-Pad1)
- Q201 pad 2: (no net) -> /Power In, Battery Charge & PV MPPT/TG1
- Q204 pad 2: (no net) -> /Power In, Battery Charge & PV MPPT/BG2
- Q205 pad 2: Net-(Q205-Pad2) -> Net-(Q205-Pad1)
- Q205 pad 3: GND -> Net-(Q205-Pad3)
- R209 pad 2: (no net) -> Net-(D201-Pad2)
- R215 pad 2: Net-(Q205-Pad2) -> Net-(Q205-Pad3)
- R217 pad 1: Net-(Q205-Pad2) -> Net-(Q205-Pad3)
- R302 pad 1: (no net) -> Net-(F301-Pad1)
- R619 pad 2: (no net) -> Net-(F601-Pad2)
- R620 pad 2: Net-(JP601-Pad1) -> Net-(P602-Pad1)
- U204 pad 25: (no net) -> Net-(R208-Pad2)
- U204 pad 32: (no net) -> Net-(R207-Pad1)
- U302 pad 24: (no net) -> Net-(P306-Pad1)
- U302 pad 28: (no net) -> Net-(U302-Pad28)
- W306 pad 1: GND -> Net-(U302-Pad28)
- W608 pad 1: Net-(JP601-Pad1) -> Net-(P602-Pad1)
Routing:
- net (no net): track 0.00 -> 63.9 mm
- net Net-(JP501-Pad1): track 41.9 -> 0.00 mm
- net +5V: track 18.1 -> 0.00 mm
- net Net-(R502-Pad2): track 3.91 -> 0.00 mm

Commit message: LTC3: Added off-board (front panel) connectors for external power and trigger circuits.
Plus an inconsequential amount of PCB layout.
Parts:
- removed M701, M702, M703, M704: W28-XQ1A-1, Oddities:Dummy_Empty
- removed P702: 43025-1000, Oddities:Dummy_Empty
- removed P704: CONN_EXT_PWR_2, Valves:VALVE-OCTAL
- removed P706: 43025-0800, Oddities:Dummy_Empty
- removed P707: CONN_EXT_PWR_3, Valves:VALVE-OCTAL
- removed P708: CONN_EXT_PWR_4, Valves:VALVE-OCTAL
- removed SW701, SW702, SW703, SW704: SP3T, Oddities:Dummy_Empty
- P703: value CONN_EXT_PWR_1 -> 43045-0800; footprint Valves:VALVE-OCTAL -> Connectors_Molex:Molex_Microfit3_Header_02x04_Angled_43045-080x
- moved R702 365.8 mm to (200.0, 161.8), turned to 270 degrees
- moved Q702 360.5 mm to (199.5, 167.7)
- moved Q701 354.9 mm to (199.5, 151.0)
- moved IC702 348.0 mm to (203.8, 162.7)
- moved C701 343.2 mm to (215.0, 152.8)
- moved R712 342.5 mm to (224.5, 171.8)
- moved R705 341.6 mm to (199.5, 155.0)
- moved R711 339.3 mm to (224.5, 155.0)
- moved R706 334.9 mm to (199.5, 171.8)
- moved R707 333.0 mm to (225.0, 145.0), turned to 270 degrees
- moved R701 331.5 mm to (200.0, 145.0), turned to 270 degrees
- moved P701 328.8 mm to (214.1, 185.7)
- moved R709 327.8 mm to (240.0, 150.0)
- moved C702 326.9 mm to (215.0, 169.5)
- moved Q704 325.8 mm to (224.5, 167.8)
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Connections:
- C703 pad 2: Net-(C703-Pad2) -> GND
- P703 pad 3: (no net) -> Net-(C702-Pad1)
- P703 pad 4: (no net) -> GND
- P703 pad 5: (no net) -> Net-(C703-Pad1)
- P703 pad 6: (no net) -> GND
- P703 pad 7: (no net) -> Net-(C704-Pad1)
- P703 pad 8: (no net) -> GND
- R709 pad 2: Net-(C703-Pad2) -> GND
Routing:
- net /External Device Power/EXT_POW_2_OPTO_RELAY_P: track 0.00 -> 31.2 mm
- net /External Device Power/EXT_POW_4_OPTO_RELAY_P: track 0.00 -> 23.4 mm
- net Net-(C704-Pad1): track 0.00 -> 6.45 mm
- net Net-(C702-Pad1): track 0.00 -> 6.45 mm
- net Net-(C701-Pad1): track 0.00 -> 6.45 mm
- net Net-(C703-Pad1): track 0.00 -> 6.19 mm
- net Net-(IC703-Pad1): track 0.00 -> 3.88 mm
- net Net-(IC701-Pad1): track 0.00 -> 3.81 mm
- net Net-(IC704-Pad1): track 0.00 -> 3.75 mm
- net Net-(IC702-Pad1): track 0.00 -> 3.75 mm
- net /GPIO_EXT_PWR_2: track 0.00 -> 3.00 mm
- net /GPIO_EXT_PWR_4: track 0.00 -> 3.00 mm
- net /GPIO_EXT_PWR_3: track 0.00 -> 3.00 mm
- net /GPIO_EXT_PWR_1: track 0.00 -> 3.00 mm

Commit message: LTC3: Layout Work
Began layout work on the power section of the LTC3.
Parts:
- moved R217 455.0 mm to (102.4, 87.4), turned to 270 degrees
- moved C206 440.0 mm to (120.6, 76.9), turned to 90 degrees
- moved R214 439.7 mm to (112.3, 85.9), turned to 180 degrees
- moved R216 436.0 mm to (105.5, 91.7), turned to 180 degrees
- moved R203 434.7 mm to (133.6, 69.7), turned to 180 degrees
- moved C218 434.0 mm to (131.0, 77.0), turned to 90 degrees
- moved R206 433.2 mm to (112.4, 73.0)
- moved R215 424.4 mm to (105.3, 83.8), turned to 270 degrees
- moved C203 421.6 mm to (120.6, 70.2), turned to 270 degrees
- moved R207 416.9 mm to (138.6, 76.1)
- moved R201 416.1 mm to (134.9, 76.9), turned to 270 degrees
- moved U204 415.0 mm to (121.8, 103.9)
- moved Q201 412.8 mm to (132.1, 86.7), turned to 90 degrees
- moved U202 412.3 mm to (112.6, 78.0)
- moved L201 411.1 mm to (144.2, 95.8)
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Routing:
- net Net-(R206-Pad1): track 0.00 -> 2.66 mm
Other:
- net class Default: clearance 0.254 -> 1; trace_width 0.254 -> 7.19
- rule trace_clearance: 0.254 -> 1
