File: ltc3/kicad/cell_protection.sch (KiCad schematic (older format))
At the start: 80 parts, among them P301 CONN_BATT_MAIN, P303 CONN_BATT_SENSE, P305 S2BPHKS, P306 PIN_HEAD_1x2, Q301 MMBT3904, Q302 SUM110P08-11, Q303 SUM110P08-11, Q304 SUM110P08-11, Q305 SUM110P08-11, Q306 NDS9407, U301 LTC2990, U302 BQ77PL900

Commit message: LTC3: Created footprint for current shunt resistor; updated schematic and PCB layout accordingly.
1. Created new footprint for Bourns CST0612 four-wire current shunt
   resistor.
2. Assigned new footprint to all current-sense resistors in schematic.
3. Created new netlist; updated PCB layout.
4. Routed DC-DC converter's shunt resistors to corresponding LTC2991
   measurement IC.
Parts:
- R302, R324: footprint Resistors_SMD:R_0805 -> LTC3:CST0612
Changed lines of the file:
@@
 F 0 "R302" V 8200 1800 50  0000 R CNN
 F 1 "30m" V 8200 2000 50  0000 L CNN
-F 2 "Resistors_SMD:R_0805" V 8030 1900 30  0001 C CNN
+F 2 "LTC3:CST0612" V 8030 1900 30  0001 C CNN
 F 3 "" H 8100 1900 30  0000 C CNN
 	1    8100 1900
@@
 F 0 "R324" V 4900 9150 50  0000 C CNN
 F 1 "1m" V 4900 8750 50  0000 C CNN
-F 2 "Resistors_SMD:R_0805" V 4780 8950 30  0001 C CNN
+F 2 "LTC3:CST0612" V 4780 8950 30  0001 C CNN
 F 3 "" H 4850 8950 30  0000 C CNN
 F 4 "1W, ±275ppm" V 4750 8950 50  0000 C CIN "Note"
