File: ltc3/kicad/charge_controller/cell_protection.sch (KiCad schematic (older format))
At the start: 80 parts, among them P301 CONN_BATT_MAIN, P303 CONN_BATT_SENSE, P305 S2BPHKS, P306 PIN_HEAD_1x2, Q301 MMBT3904, Q302 SUM110P08-11, Q303 SUM110P08-11, Q304 SUM110P08-11, Q305 SUM110P08-11, Q306 NDS9407, U301 LTC2990, U302 BQ77PL900

Commit message: LTC3: Split single-board design into two boards.
Separated the charge controller and cell protection circuitry onto its
own board (kicad/charge_controller).  The DC-DC converters,
BeagleBone, external power and triggers, and ignition fire control
circuitry remains together (kicad/ltc).

Both boards have had their schematics updated.  Sub-sheets for
circuitry moved to the other board were removed.  Still more work
remaining, though (e.g., add I2C connectors to Charge Controller
schematic; add battery power connector to LTC board; etc.).

Schematic components were *not* re-annotated to align with new sheet
numbering, as it would screw up the existing layout work (i.e., placed
components would disappear), and that would make us sad engineers.

Both boards have had their PCB layouts converted to four-layer.
Parts:
- BT301, BT302, BT303, BT304, BT305, BT306, BT307, BT308, P302, P304: footprint OFF-BOARD -> (none)
Changed lines of the file:
@@
 LIBS:741g08
 LIBS:battery_single_cell
-LIBS:BeagleBone_Black
 LIBS:bq77PL900
 LIBS:breakers
 LIBS:CD74HC14
 LIBS:current_shunt
-LIBS:EEPROMs
 LIBS:LT8490
 LIBS:LTC299x
+LIBS:MOSFET_SO8
+LIBS:MOSFET_SOT26
 LIBS:PI2127
 LIBS:PMV45EN
 LIBS:power_nodes
-LIBS:PTN78020n
 LIBS:relay_1c
 LIBS:SNx52x0
 LIBS:SUM110P08-11
 LIBS:switches2
-LIBS:MOSFET_SO8
-LIBS:MOSFET_SOT26
 LIBS:TLP
 LIBS:74xgxx
@@
 LIBS:atmel
 LIBS:audio
-LIBS:bbd
 LIBS:brooktre
 LIBS:cmos4000
@@
 LIBS:transistors
 LIBS:ttl_ieee
-LIBS:Launch_Tower_Computer_III-cache
 EELAYER 25 0
 EELAYER END
 $Descr B 17000 11000
 encoding utf-8
-Sheet 3 8
+Sheet 3 3
 Title "Battery Management"
 Date "2016-05-09"
@@
 $EndComp
 $Comp
-L GND #PWR311
+L GND #PWR056
 U 1 1 564DE030
 P 4150 8000
-F 0 "#PWR311" H 4150 7750 50  0001 C CNN
+F 0 "#PWR056" H 4150 7750 50  0001 C CNN
 F 1 "GND" H 4150 7850 50  0001 C CNN
 F 2 "" H 4150 8000 60  0000 C CNN
@@
 $EndComp
 $Comp
-L GND #PWR306
+L GND #PWR057
 U 1 1 5650209A
 P 2300 5200
-F 0 "#PWR306" H 2300 4950 50  0001 C CNN
+F 0 "#PWR057" H 2300 4950 50  0001 C CNN
 F 1 "GND" H 2300 5050 50  0001 C CNN
 F 2 "" H 2300 5200 60  0000 C CNN
@@
 $EndComp
 $Comp
-L GND #PWR301
+L GND #PWR058
 U 1 1 5650665C
 P 700 6400
-F 0 "#PWR301" H 700 6150 50  0001 C CNN
+F 0 "#PWR058" H 700 6150 50  0001 C CNN
 F 1 "GND" H 700 6250 50  0001 C CNN
 F 2 "" H 700 6400 60  0000 C CNN
@@
 $EndComp
 $Comp
-L GND #PWR303
+L GND #PWR059
 U 1 1 5652F47D
 P 1050 3000
-F 0 "#PWR303" H 1050 2750 50  0001 C CNN
+F 0 "#PWR059" H 1050 2750 50  0001 C CNN
 F 1 "GND" H 1050 2850 50  0001 C CNN
 F 2 "" H 1050 3000 60  0000 C CNN
@@
 $EndComp
 $Comp
-L VBATT #PWR302
+L VBATT #PWR060
 U 1 1 5658A738
 P 1050 1650
-F 0 "#PWR302" H 1050 1500 50  0001 C CNN
+F 0 "#PWR060" H 1050 1500 50  0001 C CNN
 F 1 "VBATT" H 1050 1800 50  0000 C CNN
 F 2 "" H 1050 1650 60  0000 C CNN
@@
 $EndComp
 $Comp
-L +5V #PWR315
+L +5V #PWR061
 U 1 1 5659CAB5
 P 14300 1000
-F 0 "#PWR315" H 14300 850 50  0001 C CNN
+F 0 "#PWR061" H 14300 850 50  0001 C CNN
 F 1 "+5V" H 14300 1140 50  0000 C CNN
 F 2 "" H 14300 1000 60  0000 C CNN
@@
 $EndComp
 $Comp
-L GND #PWR316
+L GND #PWR062
 U 1 1 5659CACB
 P 14300 2550
-F 0 "#PWR316" H 14300 2300 50  0001 C CNN
+F 0 "#PWR062" H 14300 2300 50  0001 C CNN
 F 1 "GND" H 14300 2400 50  0001 C CNN
 F 2 "" H 14300 2550 60  0000 C CNN
@@
 $EndComp
 $Comp
-L GND #PWR317
+L GND #PWR063
 U 1 1 565C67AD
 P 15200 2450
-F 0 "#PWR317" H 15200 2200 50  0001 C CNN
+F 0 "#PWR063" H 15200 2200 50  0001 C CNN
 F 1 "GND" H 15200 2300 50  0001 C CNN
 F 2 "" H 15200 2450 60  0000 C CNN
@@
 $EndComp
 $Comp
-L GND #PWR314
+L GND #PWR064
 U 1 1 565B72B8
 P 7650 3000
-F 0 "#PWR314" H 7650 2750 50  0001 C CNN
+F 0 "#PWR064" H 7650 2750 50  0001 C CNN
 F 1 "GND" H 7650 2850 50  0001 C CNN
 F 2 "" H 7650 3000 60  0000 C CNN
@@
 $EndComp
 $Comp
-L GND #PWR310
+L GND #PWR065
 U 1 1 565D2BB8
 P 3700 4900
-F 0 "#PWR310" H 3700 4650 50  0001 C CNN
+F 0 "#PWR065" H 3700 4650 50  0001 C CNN
 F 1 "GND" H 3700 4750 50  0001 C CNN
 F 2 "" H 3700 4900 60  0000 C CNN
@@
 $EndComp
 $Comp
-L GND #PWR308
+L GND #PWR066
 U 1 1 565F5A93
 P 2675 7050
-F 0 "#PWR308" H 2675 6800 50  0001 C CNN
+F 0 "#PWR066" H 2675 6800 50  0001 C CNN
 F 1 "GND" H 2675 6900 50  0001 C CNN
 F 2 "" H 2675 7050 60  0000 C CNN
@@
 $EndComp
 $Comp
-L GND #PWR304
+L GND #PWR067
 U 1 1 565FA5A2
 P 1300 7100
-F 0 "#PWR304" H 1300 6850 50  0001 C CNN
+F 0 "#PWR067" H 1300 6850 50  0001 C CNN
 F 1 "GND" H 1300 6950 50  0001 C CNN
 F 2 "" H 1300 7100 60  0000 C CNN
@@
 $EndComp
 $Comp
-L GND #PWR312
+L GND #PWR068
 U 1 1 565E5619
 P 4550 9200
-F 0 "#PWR312" H 4550 8950 50  0001 C CNN
+F 0 "#PWR068" H 4550 8950 50  0001 C CNN
 F 1 "GND" H 4550 9050 50  0001 C CNN
 F 2 "" H 4550 9200 60  0000 C CNN
@@
 F 0 "P304" H 10350 6750 50  0000 C CNN
 F 1 "~" V 10450 6300 50  0000 C CNN
-F 2 "OFF-BOARD" H 10350 6300 60  0001 C CNN
+F 2 "" H 10350 6300 60  0001 C CNN
 F 3 "" H 10350 6300 60  0000 C CNN
 	1    10350 6300
@@
 F 0 "P302" H 10350 5200 50  0000 C CNN
 F 1 "~" V 10450 5050 50  0000 C CNN
-F 2 "OFF-BOARD" H 10350 5050 60  0001 C CNN
+F 2 "" H 10350 5050 60  0001 C CNN
 F 3 "" H 10350 5050 60  0000 C CNN
 	1    10350 5050
@@
 F 0 "BT301" H 11418 5850 50  0000 L CNN
 F 1 "~" H 11418 5804 50  0000 L CNN
-F 2 "OFF-BOARD" V 11300 5860 60  0001 C CNN
+F 2 "" V 11300 5860 60  0001 C CNN
 F 3 "" V 11300 5860 60  0000 C CNN
 	1    11300 5850
@@
 F 0 "BT302" H 11418 6250 50  0000 L CNN
 F 1 "~" H 11418 6204 50  0000 L CNN
-F 2 "OFF-BOARD" V 11300 6260 60  0001 C CNN
+F 2 "" V 11300 6260 60  0001 C CNN
 F 3 "" V 11300 6260 60  0000 C CNN
 	1    11300 6250
@@
 F 0 "BT303" H 11418 6650 50  0000 L CNN
 F 1 "~" H 11418 6604 50  0000 L CNN
-F 2 "OFF-BOARD" V 11300 6660 60  0001 C CNN
+F 2 "" V 11300 6660 60  0001 C CNN
 F 3 "" V 11300 6660 60  0000 C CNN
 	1    11300 6650
@@
 F 0 "BT304" H 11418 7050 50  0000 L CNN
 F 1 "~" H 11418 7004 50  0000 L CNN
-F 2 "OFF-BOARD" V 11300 7060 60  0001 C CNN
+F 2 "" V 11300 7060 60  0001 C CNN
 F 3 "" V 11300 7060 60  0000 C CNN
 	1    11300 7050
@@
 F 0 "BT305" H 11418 7450 50  0000 L CNN
 F 1 "~" H 11418 7404 50  0000 L CNN
-F 2 "OFF-BOARD" V 11300 7460 60  0001 C CNN
+F 2 "" V 11300 7460 60  0001 C CNN
 F 3 "" V 11300 7460 60  0000 C CNN
 	1    11300 7450
@@
 F 0 "BT306" H 11418 7850 50  0000 L CNN
 F 1 "~" H 11418 7804 50  0000 L CNN
-F 2 "OFF-BOARD" V 11300 7860 60  0001 C CNN
+F 2 "" V 11300 7860 60  0001 C CNN
 F 3 "" V 11300 7860 60  0000 C CNN
 	1    11300 7850
@@
 F 0 "BT307" H 11418 8250 50  0000 L CNN
 F 1 "~" H 11418 8204 50  0000 L CNN
-F 2 "OFF-BOARD" V 11300 8260 60  0001 C CNN
+F 2 "" V 11300 8260 60  0001 C CNN
 F 3 "" V 11300 8260 60  0000 C CNN
 	1    11300 8250
@@
 F 0 "BT308" H 11418 8650 50  0000 L CNN
 F 1 "~" H 11418 8604 50  0000 L CNN
-F 2 "OFF-BOARD" V 11300 8660 60  0001 C CNN
+F 2 "" V 11300 8660 60  0001 C CNN
 F 3 "" V 11300 8660 60  0000 C CNN
 	1    11300 8650
@@
 $EndComp
 $Comp
-L GND #PWR313
+L GND #PWR069
 U 1 1 56CBF3B2
 P 5550 4650
-F 0 "#PWR313" H 5550 4400 50  0001 C CNN
+F 0 "#PWR069" H 5550 4400 50  0001 C CNN
 F 1 "GND" H 5550 4500 50  0001 C CNN
 F 2 "" H 5550 4650 60  0000 C CNN
@@
 $EndComp
 $Comp
-L GND #PWR307
+L GND #PWR070
 U 1 1 56E4B689
 P 2500 7750
-F 0 "#PWR307" H 2500 7500 50  0001 C CNN
+F 0 "#PWR070" H 2500 7500 50  0001 C CNN
 F 1 "GND" H 2500 7600 50  0001 C CNN
 F 2 "" H 2500 7750 60  0000 C CNN
@@
 $EndComp
 $Comp
-L GND #PWR309
+L GND #PWR071
 U 1 1 56E4A519
 P 3100 7750
-F 0 "#PWR309" H 3100 7500 50  0001 C CNN
+F 0 "#PWR071" H 3100 7500 50  0001 C CNN
 F 1 "GND" H 3108 7577 50  0001 C CNN
 F 2 "" H 3100 7750 50  0000 C CNN
@@
 Connection ~ 2100 2450
 $Comp
-L GND #PWR305
+L GND #PWR072
 U 1 1 573455B4
 P 2100 3100
-F 0 "#PWR305" H 2100 2850 50  0001 C CNN
+F 0 "#PWR072" H 2100 2850 50  0001 C CNN
 F 1 "GND" H 2105 2927 50  0000 C CNN
 F 2 "" H 2100 3100 50  0000 C CNN
