File: ltc3/kicad/cell_protection/LTC3_Cell_Protection.sch (KiCad schematic (older format))
At the start: 82 parts, among them P1 S2BPHKS, P2 PIN_HEAD_1x2, P3 MicroFit header, P4 XH header, straight, P7 MicroFit head., P8 MicroFit head., Q1 SUM110P08-11, Q2 SUM110P08-11, Q3 NDS9407, Q4 SUM110P08-11, Q5 SUM110P08-11, Q6 MMBT3904, U1 BQ77PL900, U2 LTC2990

Commit message: LTC3: Layout Work/Connector Updating
Added many needed connectors and added to layout.

	-Added 5V nodes for Charge Controller/Cell Protection
	-Added I2C bus connectors
	-Added Vin connectors for Cell Protection

Added all connectors to layout and ensured all nodes were connected.
Parts:
- added P9: XH header, straight, Connectors_JST:JST_XH_B02B-XH-A_02x2.50mm_Straight, symbol CONN_01X02
Connections:
- net +5V: now also C1.1, U1.32 (VLOG), U1.34 (CNF1), U1.42 (VREG1)
- net I2C_DATA: now also U2.7 (SDL), P9.1 (P1); no longer U2.6 (SDA)
- net I2C_CLOCK renamed I2C_CLK
- net I2C_CLK: now also U2.6 (SDA), P9.2 (P2); no longer U2.7 (SDL)
Changed lines of the file:
@@
 LIBS:atmel
 LIBS:audio
+LIBS:bbd
 LIBS:brooktre
 LIBS:cmos4000
@@
 $EndComp
 $Comp
-L GND #PWR16
+L GND #PWR12
 U 1 1 564DE030
 P 4550 8000
-F 0 "#PWR16" H 4550 7750 50  0001 C CNN
+F 0 "#PWR12" H 4550 7750 50  0001 C CNN
 F 1 "GND" H 4550 7850 50  0001 C CNN
 F 2 "" H 4550 8000 60  0000 C CNN
@@
 $EndComp
 $Comp
-L GND #PWR10
+L GND #PWR7
 U 1 1 5650209A
 P 2700 5200
-F 0 "#PWR10" H 2700 4950 50  0001 C CNN
+F 0 "#PWR7" H 2700 4950 50  0001 C CNN
 F 1 "GND" H 2700 5050 50  0001 C CNN
 F 2 "" H 2700 5200 60  0000 C CNN
@@
 $EndComp
 $Comp
-L GND #PWR11
+L GND #PWR2
 U 1 1 5650665C
 P 1100 6400
-F 0 "#PWR11" H 1100 6150 50  0001 C CNN
+F 0 "#PWR2" H 1100 6150 50  0001 C CNN
 F 1 "GND" H 1100 6250 50  0001 C CNN
 F 2 "" H 1100 6400 60  0000 C CNN
@@
 Text HLabel 3500 6400 0    50   3State ~ 0
 BQ_XALERT
-Text HLabel 3500 6200 0    50   3State ~ 0
-I2C_DATA
-Text HLabel 3500 6300 0    50   3State ~ 0
-I2C_CLOCK
 Text Notes 3400 5550 2    50   Italic 0
 5.0VDC
@@
 $EndComp
 $Comp
-L GND #PWR5
+L GND #PWR4
 U 1 1 5652F47D
 P 1450 3000
-F 0 "#PWR5" H 1450 2750 50  0001 C CNN
+F 0 "#PWR4" H 1450 2750 50  0001 C CNN
 F 1 "GND" H 1450 2850 50  0001 C CNN
 F 2 "" H 1450 3000 60  0000 C CNN
@@
 $EndComp
 $Comp
-L +5V #PWR1
+L +5V #PWR16
 U 1 1 5659CAB5
 P 14300 1000
-F 0 "#PWR1" H 14300 850 50  0001 C CNN
+F 0 "#PWR16" H 14300 850 50  0001 C CNN
 F 1 "+5V" H 14300 1140 50  0000 C CNN
 F 2 "" H 14300 1000 60  0000 C CNN
@@
 	1    0    0    -1
 $EndComp
-Text HLabel 15650 1900 2    50   BiDi ~ 0
-I2C_CLOCK
-Text HLabel 15650 2000 2    50   BiDi ~ 0
-I2C_DATA
 Text Notes 11400 2750 0    50   Italic 0
 I2C addr 0x9A
@@
 $EndComp
 $Comp
-L GND #PWR4
+L GND #PWR17
 U 1 1 5659CACB
 P 14300 2550
-F 0 "#PWR4" H 14300 2300 50  0001 C CNN
+F 0 "#PWR17" H 14300 2300 50  0001 C CNN
 F 1 "GND" H 14300 2400 50  0001 C CNN
 F 2 "" H 14300 2550 60  0000 C CNN
@@
 $EndComp
 $Comp
-L GND #PWR3
+L GND #PWR18
 U 1 1 565C67AD
 P 15200 2450
-F 0 "#PWR3" H 15200 2200 50  0001 C CNN
+F 0 "#PWR18" H 15200 2200 50  0001 C CNN
 F 1 "GND" H 15200 2300 50  0001 C CNN
 F 2 "" H 15200 2450 60  0000 C CNN
@@
 $EndComp
 $Comp
-L GND #PWR6
+L GND #PWR15
 U 1 1 565B72B8
 P 8050 3000
-F 0 "#PWR6" H 8050 2750 50  0001 C CNN
+F 0 "#PWR15" H 8050 2750 50  0001 C CNN
 F 1 "GND" H 8050 2850 50  0001 C CNN
 F 2 "" H 8050 3000 60  0000 C CNN
@@
 $EndComp
 $Comp
-L GND #PWR9
+L GND #PWR11
 U 1 1 565D2BB8
 P 4100 4900
-F 0 "#PWR9" H 4100 4650 50  0001 C CNN
+F 0 "#PWR11" H 4100 4650 50  0001 C CNN
 F 1 "GND" H 4100 4750 50  0001 C CNN
 F 2 "" H 4100 4900 60  0000 C CNN
@@
 $EndComp
 $Comp
-L GND #PWR12
+L GND #PWR9
 U 1 1 565F5A93
 P 3075 7050
-F 0 "#PWR12" H 3075 6800 50  0001 C CNN
+F 0 "#PWR9" H 3075 6800 50  0001 C CNN
 F 1 "GND" H 3075 6900 50  0001 C CNN
 F 2 "" H 3075 7050 60  0000 C CNN
@@
 $EndComp
 $Comp
-L GND #PWR13
+L GND #PWR5
 U 1 1 565FA5A2
 P 1700 7100
-F 0 "#PWR13" H 1700 6850 50  0001 C CNN
+F 0 "#PWR5" H 1700 6850 50  0001 C CNN
 F 1 "GND" H 1700 6950 50  0001 C CNN
 F 2 "" H 1700 7100 60  0000 C CNN
@@
 $EndComp
 $Comp
-L GND #PWR17
+L GND #PWR13
 U 1 1 565E5619
 P 4950 9200
-F 0 "#PWR17" H 4950 8950 50  0001 C CNN
+F 0 "#PWR13" H 4950 8950 50  0001 C CNN
 F 1 "GND" H 4950 9050 50  0001 C CNN
 F 2 "" H 4950 9200 60  0000 C CNN
@@
 $EndComp
 $Comp
-L GND #PWR8
+L GND #PWR14
 U 1 1 56CBF3B2
 P 5950 4650
-F 0 "#PWR8" H 5950 4400 50  0001 C CNN
+F 0 "#PWR14" H 5950 4400 50  0001 C CNN
 F 1 "GND" H 5950 4500 50  0001 C CNN
 F 2 "" H 5950 4650 60  0000 C CNN
@@
 $EndComp
 $Comp
-L GND #PWR14
+L GND #PWR8
 U 1 1 56E4B689
 P 2900 7750
-F 0 "#PWR14" H 2900 7500 50  0001 C CNN
+F 0 "#PWR8" H 2900 7500 50  0001 C CNN
 F 1 "GND" H 2900 7600 50  0001 C CNN
 F 2 "" H 2900 7750 60  0000 C CNN
@@
 $EndComp
 $Comp
-L GND #PWR15
+L GND #PWR10
 U 1 1 56E4A519
 P 3500 7750
-F 0 "#PWR15" H 3500 7500 50  0001 C CNN
+F 0 "#PWR10" H 3500 7500 50  0001 C CNN
 F 1 "GND" H 3508 7577 50  0001 C CNN
 F 2 "" H 3500 7750 50  0000 C CNN
@@
 Connection ~ 3600 5550
 Wire Wire Line
-	1100 5800 1100 5550
+	1100 5400 1100 5800
 Wire Wire Line
 	1100 5550 3750 5550
@@
 Connection ~ 2500 2450
 $Comp
-L GND #PWR7
+L GND #PWR6
 U 1 1 573455B4
 P 2500 3100
-F 0 "#PWR7" H 2500 2850 50  0001 C CNN
+F 0 "#PWR6" H 2500 2850 50  0001 C CNN
 F 1 "GND" H 2505 2927 50  0000 C CNN
 F 2 "" H 2500 3100 50  0000 C CNN
@@
 VBATT
 $Comp
-L GND #PWR2
+L GND #PWR3
 U 1 1 579182C2
 P 1200 1900
-F 0 "#PWR2" H 1200 1650 50  0001 C CNN
+F 0 "#PWR3" H 1200 1650 50  0001 C CNN
 F 1 "GND" H 1200 1750 50  0000 C CNN
 F 2 "" H 1200 1900 50  0000 C CNN
@@
 	1050 1650 1450 1650
 Connection ~ 1450 1650
+Connection ~ 1100 5550
+$Comp
+L +5V #PWR1
+U 1 1 578B2BD9
+P 1100 5400
+F 0 "#PWR1" H 1100 5250 50  0001 C CNN
+F 1 "+5V" H 1115 5573 50  0000 C CNN
+F 2 "" H 1100 5400 50  0000 C CNN
+F 3 "" H 1100 5400 50  0000 C CNN
+	1    1100 5400
+	1    0    0    -1
+$EndComp
+$Comp
+L CONN_01X02 P9
+U 1 1 578C7D35
+P 15850 1950
+F 0 "P9" H 15850 2400 50  0000 C CNN
+F 1 "XH header, straight" V 15950 1950 50  0000 C CNN
+F 2 "Connectors_JST:JST_XH_B02B-XH-A_02x2.50mm_Straight" H 15850 1950 60  0001 C CNN
+F 3 "http://www.jst-mfg.com/product/pdf/eng/eXH.pdf" H 15850 1950 60  0001 C CNN
+F 4 "-" H 15850 1950 60  0001 C CNN "Spec"
+F 5 "TO LTC" V 16050 1950 50  0000 C CIN "Note"
+F 6 "JST" H 15850 1950 60  0001 C CNN "Mfg_Name"
+F 7 "B2B-XH-A" H 15850 1950 60  0001 C CNN "Mfg_PN"
+	1    15850 1950
+	1    0    0    -1
+$EndComp
+Text Label 3500 6200 0    41   ~ 0
+I2C_DATA
+Text Label 3500 6300 0    41   ~ 0
+I2C_CLK
+Wire Wire Line
+	15450 1900 15450 2450
+Connection ~ 15450 1900
+Wire Wire Line
+	15600 2000 15600 2450
+Connection ~ 15600 2000
+Text Label 15450 2450 1    80   ~ 0
+I2C_DATA
+Text Label 15600 2450 1    80   ~ 0
+I2C_CLK
 $EndSCHEMATC

Commit message: LTC3: Layout Review Notes
Had a layout review this morning (hooray!) and added "TODO" notes to all
the boards and schematics.  More work to be done!
Other:
- note added: "CHANGE THIS GROUND TO BE DIFF FROM BOARD GND"
- note added: "Goodbye"
- note added: "Move away from output to input"
- note added: "change connector to 4 pin w/5v/Gnd"
Changed lines of the file:
@@
 LIBS:breakers
 LIBS:CD74HC14
-LIBS:current_shunt
 LIBS:LT8490
 LIBS:LTC299x
@@
 Text Label 15600 2450 1    80   ~ 0
 I2C_CLK
+Text Notes 15800 2200 0    80   ~ 0
+change connector to 4 pin w/5v/Gnd
+Text Notes 13450 2750 0    80   ~ 0
+CHANGE THIS GROUND TO BE DIFF FROM BOARD GND
+Text Notes 8450 2100 0    80   ~ 0
+Move away from output to input
+Text Notes 1000 5200 0    80   ~ 0
+Goodbye
 $EndSCHEMATC
