File: ltc3/kicad/ltc/beaglebone_cape.sch (KiCad schematic (older format))
At the start: 13 parts, among them P301 BeagleBone_Black_Expansion_He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, P302 BeagleBone_Black_Expansion_He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, P303 JST PH header, P304 JST PH header, U301 CAT24C256

Commit message: LTC3: More BOM work, mostly on the LTC proper.
Plus a few minor tweaks to the charge controller and cell protection
BOMs that should not impact PCB layout.

Nearly finished with LTC BOM.
Parts:
- C301: Mfg_Description (none) -> 100V X7R 10%; Mfg_Name - -> Murata; Mfg_PN - -> GCM21BR72A104KA37L
- JP301: Mfg_Description (none) -> -; Mfg_Name (none) -> -; Mfg_PN (none) -> -; Note (none) -> Pin Header, 1x2; Spec (none) -> -
- P301, P302, W301, W302: Mfg_Description (none) -> -; Mfg_Name (none) -> -; Mfg_PN (none) -> -; Note (none) -> -; Spec (none) -> -
- P303, P304: Mfg_Description (none) -> -
- R301, R302, R303, R304: footprint Resistors_SMD:R_0603 -> Resistors_SMD:R_0805; Mfg_Description (none) -> 1% 1/8W; Mfg_Name - -> Yageo; Mfg_PN - -> RC0805FR-075K6L
- U301: Mfg_Description (none) -> EEPROM 256KBIT 400KHZ
