File: ltc3/kicad/ltc/dcdc_converter.sch (KiCad schematic (older format))
At the start: 41 parts, among them P401 43045-1000, P402 43025-1000, Q401 BSS138, Q402 BSS138, Q403 BSS138, SW401 SPDT, SW402 SP3T, SW403 SP3T, U401 PTN78020W, U402 LTC2991, U403 PTN78020H, U404 PTN78020H

Commit message: LTC3: Split single-board design into two boards.
Separated the charge controller and cell protection circuitry onto its
own board (kicad/charge_controller).  The DC-DC converters,
BeagleBone, external power and triggers, and ignition fire control
circuitry remains together (kicad/ltc).

Both boards have had their schematics updated.  Sub-sheets for
circuitry moved to the other board were removed.  Still more work
remaining, though (e.g., add I2C connectors to Charge Controller
schematic; add battery power connector to LTC board; etc.).

Schematic components were *not* re-annotated to align with new sheet
numbering, as it would screw up the existing layout work (i.e., placed
components would disappear), and that would make us sad engineers.

Both boards have had their PCB layouts converted to four-layer.
Parts:
- P402, SW401, SW402, SW403: footprint OFF-BOARD -> (none)
Changed lines of the file:
@@
 LIBS:atmel
 LIBS:audio
-LIBS:bbd
 LIBS:brooktre
 LIBS:cmos4000
@@
 LIBS:transistors
 LIBS:ttl_ieee
-LIBS:Launch_Tower_Computer_III-cache
 EELAYER 25 0
 EELAYER END
 $Descr B 17000 11000
 encoding utf-8
-Sheet 4 8
+Sheet 4 6
 Title "LTC3 DC-DC Converters"
 Date "2016-05-09"
@@
 $EndDescr
 $Comp
-L GND #PWR407
+L GND #PWR01
 U 1 1 5557F6A3
 P 2650 1900
-F 0 "#PWR407" H 2650 1900 30  0001 C CNN
+F 0 "#PWR01" H 2650 1900 30  0001 C CNN
 F 1 "GND" H 2650 1830 30  0001 C CNN
 F 2 "" H 2650 1900 60  0000 C CNN
@@
 $EndComp
 $Comp
-L GND #PWR413
+L GND #PWR02
 U 1 1 5557F6B2
 P 5050 1900
-F 0 "#PWR413" H 5050 1900 30  0001 C CNN
+F 0 "#PWR02" H 5050 1900 30  0001 C CNN
 F 1 "GND" H 5050 1830 30  0001 C CNN
 F 2 "" H 5050 1900 60  0000 C CNN
@@
 $EndComp
 $Comp
-L GND #PWR416
+L GND #PWR03
 U 1 1 5557F6ED
 P 5250 2100
-F 0 "#PWR416" H 5250 2100 30  0001 C CNN
+F 0 "#PWR03" H 5250 2100 30  0001 C CNN
 F 1 "GND" H 5250 2030 30  0001 C CNN
 F 2 "" H 5250 2100 60  0000 C CNN
@@
 $EndComp
 $Comp
-L GND #PWR404
+L GND #PWR04
 U 1 1 5557F71B
 P 2250 2100
-F 0 "#PWR404" H 2250 2100 30  0001 C CNN
+F 0 "#PWR04" H 2250 2100 30  0001 C CNN
 F 1 "GND" H 2250 2030 30  0001 C CNN
 F 2 "" H 2250 2100 60  0000 C CNN
@@
 $EndComp
 $Comp
-L GND #PWR408
+L GND #PWR05
 U 1 1 55945CE3
 P 2650 5150
-F 0 "#PWR408" H 2650 5150 30  0001 C CNN
+F 0 "#PWR05" H 2650 5150 30  0001 C CNN
 F 1 "GND" H 2650 5080 30  0001 C CNN
 F 2 "" H 2650 5150 60  0000 C CNN
@@
 $EndComp
 $Comp
-L GND #PWR414
+L GND #PWR06
 U 1 1 55945CE9
 P 5050 5150
-F 0 "#PWR414" H 5050 5150 30  0001 C CNN
+F 0 "#PWR06" H 5050 5150 30  0001 C CNN
 F 1 "GND" H 5050 5080 30  0001 C CNN
 F 2 "" H 5050 5150 60  0000 C CNN
@@
 $EndComp
 $Comp
-L GND #PWR417
+L GND #PWR07
 U 1 1 55945CFE
 P 5250 5350
-F 0 "#PWR417" H 5250 5350 30  0001 C CNN
+F 0 "#PWR07" H 5250 5350 30  0001 C CNN
 F 1 "GND" H 5250 5280 30  0001 C CNN
 F 2 "" H 5250 5350 60  0000 C CNN
@@
 $EndComp
 $Comp
-L GND #PWR405
+L GND #PWR08
 U 1 1 55945D0D
 P 2250 5350
-F 0 "#PWR405" H 2250 5350 30  0001 C CNN
+F 0 "#PWR08" H 2250 5350 30  0001 C CNN
 F 1 "GND" H 2250 5280 30  0001 C CNN
 F 2 "" H 2250 5350 60  0000 C CNN
@@
 $EndComp
 $Comp
-L GND #PWR409
+L GND #PWR09
 U 1 1 55946855
 P 2650 8550
-F 0 "#PWR409" H 2650 8550 30  0001 C CNN
+F 0 "#PWR09" H 2650 8550 30  0001 C CNN
 F 1 "GND" H 2650 8480 30  0001 C CNN
 F 2 "" H 2650 8550 60  0000 C CNN
@@
 $EndComp
 $Comp
-L GND #PWR415
+L GND #PWR010
 U 1 1 5594685B
 P 5050 8550
-F 0 "#PWR415" H 5050 8550 30  0001 C CNN
+F 0 "#PWR010" H 5050 8550 30  0001 C CNN
 F 1 "GND" H 5050 8480 30  0001 C CNN
 F 2 "" H 5050 8550 60  0000 C CNN
@@
 $EndComp
 $Comp
-L GND #PWR418
+L GND #PWR011
 U 1 1 5594686D
 P 5250 8750
-F 0 "#PWR418" H 5250 8750 30  0001 C CNN
+F 0 "#PWR011" H 5250 8750 30  0001 C CNN
 F 1 "GND" H 5250 8680 30  0001 C CNN
 F 2 "" H 5250 8750 60  0000 C CNN
@@
 $EndComp
 $Comp
-L GND #PWR412
+L GND #PWR012
 U 1 1 5594688C
 P 3850 9800
-F 0 "#PWR412" H 3850 9550 50  0001 C CNN
+F 0 "#PWR012" H 3850 9550 50  0001 C CNN
 F 1 "GND" H 3850 9650 50  0001 C CNN
 F 2 "" H 3850 9800 60  0000 C CNN
@@
 $EndComp
 $Comp
-L GND #PWR406
+L GND #PWR013
 U 1 1 5594B465
 P 2250 8750
-F 0 "#PWR406" H 2250 8750 30  0001 C CNN
+F 0 "#PWR013" H 2250 8750 30  0001 C CNN
 F 1 "GND" H 2250 8680 30  0001 C CNN
 F 2 "" H 2250 8750 60  0000 C CNN
@@
 $EndComp
 $Comp
-L +5V #PWR419
+L +5V #PWR014
 U 1 1 56538996
 P 6650 1100
-F 0 "#PWR419" H 6650 950 50  0001 C CNN
+F 0 "#PWR014" H 6650 950 50  0001 C CNN
 F 1 "+5V" H 6650 1240 50  0000 C CNN
 F 2 "" H 6650 1100 60  0000 C CNN
@@
 $EndComp
 $Comp
-L VBATT #PWR403
+L VBATT #PWR015
 U 1 1 565394B2
 P 1600 1100
-F 0 "#PWR403" H 1600 950 50  0001 C CNN
+F 0 "#PWR015" H 1600 950 50  0001 C CNN
 F 1 "VBATT" H 1600 1250 50  0000 C CNN
 F 2 "" H 1600 1100 60  0000 C CNN
@@
 $EndComp
 $Comp
-L VBATT #PWR401
+L VBATT #PWR016
 U 1 1 5653A057
 P 1150 4350
-F 0 "#PWR401" H 1150 4200 50  0001 C CNN
+F 0 "#PWR016" H 1150 4200 50  0001 C CNN
 F 1 "VBATT" H 1150 4500 50  0000 C CNN
 F 2 "" H 1150 4350 60  0000 C CNN
@@
 $EndComp
 $Comp
-L +12V #PWR421
+L +12V #PWR017
 U 1 1 5653A6FD
 P 6650 4350
-F 0 "#PWR421" H 6650 4200 50  0001 C CNN
+F 0 "#PWR017" H 6650 4200 50  0001 C CNN
 F 1 "+12V" H 6650 4490 50  0000 C CNN
 F 2 "" H 6650 4350 60  0000 C CNN
@@
 $EndComp
 $Comp
-L VBATT #PWR402
+L VBATT #PWR018
 U 1 1 5653ADB9
 P 1150 7750
-F 0 "#PWR402" H 1150 7600 50  0001 C CNN
+F 0 "#PWR018" H 1150 7600 50  0001 C CNN
 F 1 "VBATT" H 1150 7900 50  0000 C CNN
 F 2 "" H 1150 7750 60  0000 C CNN
@@
 $EndComp
 $Comp
-L +19V #PWR423
+L +19V #PWR019
 U 1 1 5653B5C8
 P 6650 7600
-F 0 "#PWR423" H 6650 7450 50  0001 C CNN
+F 0 "#PWR019" H 6650 7450 50  0001 C CNN
 F 1 "+19V" H 6650 7740 50  0000 C CNN
 F 2 "" H 6650 7600 60  0000 C CNN
@@
 $EndComp
 $Comp
-L +5V #PWR427
+L +5V #PWR020
 U 1 1 56588D70
 P 14350 1100
-F 0 "#PWR427" H 14350 950 50  0001 C CNN
+F 0 "#PWR020" H 14350 950 50  0001 C CNN
 F 1 "+5V" H 14350 1240 50  0000 C CNN
 F 2 "" H 14350 1100 60  0000 C CNN
@@
 +19V DC Supply
 $Comp
-L GND #PWR428
+L GND #PWR021
 U 1 1 565F268D
 P 14350 3000
-F 0 "#PWR428" H 14350 2750 50  0001 C CNN
+F 0 "#PWR021" H 14350 2750 50  0001 C CNN
 F 1 "GND" H 14350 2850 50  0001 C CNN
 F 2 "" H 14350 3000 60  0000 C CNN
@@
 $EndComp
 $Comp
-L GND #PWR424
+L GND #PWR022
 U 1 1 56C97D65
 P 6650 9000
-F 0 "#PWR424" H 6650 8750 50  0001 C CNN
+F 0 "#PWR022" H 6650 8750 50  0001 C CNN
 F 1 "GND" H 6650 8850 50  0001 C CNN
 F 2 "" H 6650 9000 50  0000 C CNN
@@
 $EndComp
 $Comp
-L GND #PWR422
+L GND #PWR023
 U 1 1 56C983B8
 P 6650 5600
-F 0 "#PWR422" H 6650 5350 50  0001 C CNN
+F 0 "#PWR023" H 6650 5350 50  0001 C CNN
 F 1 "GND" H 6650 5450 50  0001 C CNN
 F 2 "" H 6650 5600 50  0000 C CNN
@@
 $EndComp
 $Comp
-L GND #PWR420
+L GND #PWR024
 U 1 1 56C98C65
 P 6650 2350
-F 0 "#PWR420" H 6650 2100 50  0001 C CNN
+F 0 "#PWR024" H 6650 2100 50  0001 C CNN
 F 1 "GND" H 6650 2200 50  0001 C CNN
 F 2 "" H 6650 2350 50  0000 C CNN
@@
 Manual Override Switches, Front Panel
 $Comp
-L GND #PWR426
+L GND #PWR025
 U 1 1 57289E82
 P 12700 6050
-F 0 "#PWR426" H 12700 5800 50  0001 C CNN
+F 0 "#PWR025" H 12700 5800 50  0001 C CNN
 F 1 "GND" H 12708 5876 50  0001 C CNN
 F 2 "" H 12700 6050 50  0000 C CNN
@@
 F 0 "SW402" V 15100 6100 50  0000 R CNN
 F 1 "SP3T" V 15200 6100 50  0000 R CNN
-F 2 "OFF-BOARD" H 14575 6325 50  0001 C CNN
+F 2 "" H 14575 6325 50  0001 C CNN
 F 3 "" H 14575 6325 50  0000 C CNN
 	1    15200 6150
@@
 F 0 "SW403" V 15750 6100 50  0000 R CNN
 F 1 "SP3T" V 15850 6100 50  0000 R CNN
-F 2 "OFF-BOARD" H 15225 6325 50  0001 C CNN
+F 2 "" H 15225 6325 50  0001 C CNN
 F 3 "" H 15225 6325 50  0000 C CNN
 	1    15850 6150
@@
 $EndComp
 $Comp
-L GND #PWR411
+L GND #PWR026
 U 1 1 572980E2
 P 3850 6400
-F 0 "#PWR411" H 3850 6150 50  0001 C CNN
+F 0 "#PWR026" H 3850 6150 50  0001 C CNN
 F 1 "GND" H 3850 6250 50  0001 C CNN
 F 2 "" H 3850 6400 60  0000 C CNN
@@
 $EndComp
 $Comp
-L GND #PWR410
+L GND #PWR027
 U 1 1 5729A826
 P 3850 3150
-F 0 "#PWR410" H 3850 2900 50  0001 C CNN
+F 0 "#PWR027" H 3850 2900 50  0001 C CNN
 F 1 "GND" H 3850 3000 50  0001 C CNN
 F 2 "" H 3850 3150 60  0000 C CNN
@@
 F 0 "SW401" V 14450 6100 50  0000 R CNN
 F 1 "SPDT" V 14550 6100 50  0000 R CNN
-F 2 "OFF-BOARD" H 14550 6150 60  0001 C CNN
+F 2 "" H 14550 6150 60  0001 C CNN
 F 3 "" H 14550 6150 60  0000 C CNN
 	1    14550 6150
@@
 F 0 "P402" H 13800 6000 50  0000 L CNN
 F 1 "43025-1000" V 13900 4950 50  0000 L CNN
-F 2 "OFF-BOARD" H 13800 5450 50  0001 C CNN
+F 2 "" H 13800 5450 50  0001 C CNN
 F 3 "" H 13800 5450 50  0000 C CNN
 F 4 "MicroFit3 2x5 recept." V 14000 4950 50  0000 L CNN "Note"
@@
 Connection ~ 12700 5400
 $Comp
-L +3.3V #PWR425
+L +3.3V #PWR028
 U 1 1 5728FE05
 P 12700 4850
-F 0 "#PWR425" H 12700 4700 50  0001 C CNN
+F 0 "#PWR028" H 12700 4700 50  0001 C CNN
 F 1 "+3.3V" H 12715 5023 50  0000 C CNN
 F 2 "" H 12700 4850 50  0000 C CNN

Commit message: LTC3: Updates to LTC schematic.
1. Cleaned up top-level sheet.
2. Added board-to-board connectors for power, I2C.
3. Miscelleneous component part selection/changes.
Parts:
- removed C407, C408, C409, C412, C413, C414, C415: 4.7μ, Capacitors_SMD:C_0805, symbol C
- removed C410, C416: 470μ, Capacitors_ThroughHole:C_Radial_D10_L25_P5, symbol CP1
- removed C411, C417: 1μ, Capacitors_SMD:C_0805, symbol C
- removed Q402, Q403: BSS138, TO_SOT_Packages_SMD:SOT-23, symbol Q_NMOS_GSD
- removed R401: 0.1, LTC3:CST0612, symbol R4T
- removed R403, R405: 60m, LTC3:CST0612, symbol R4T
- removed R406: 2.91k, Resistors_SMD:R_0805, symbol R
- added C207, C208, C209, C212, C213, C214, C215: 4.7μ, Capacitors_SMD:C_0805, symbol C
- added C210, C216: 470μ, Capacitors_ThroughHole:C_Radial_D10_L25_P5, symbol C
- added C211, C217: 1μ, Capacitors_SMD:C_0805, symbol C
- added P201: MicroFit header, Connectors_Molex:Molex_Microfit3_Header_02x01_Straight_43045-0228, symbol CONN_01X02
- added Q202, Q203: BSS138, TO_SOT_Packages_SMD:SOT-23, symbol Q_NMOS_GSD
- added R201, R203, R205: 60m, LTC3:CST0612, symbol R4T
- added R206: 2.91k, Resistors_SMD:R_0805, symbol R
- C201: renamed from C402; Mfg_Name (none) -> -; Mfg_PN (none) -> -; Note (none) -> -; Spec (none) -> 75V
- C202: renamed from C403; Mfg_Name (none) -> -; Mfg_PN (none) -> -; Note ceramic, X[57]R -> -; Spec (none) -> 75V X7R
- C203: renamed from C404; symbol CP1 -> C; Mfg_Name (none) -> -; Mfg_PN (none) -> -; Note (none) -> -; Spec (none) -> 75V
- C204: renamed from C405; Mfg_Name (none) -> -; Mfg_PN (none) -> -; Note (none) -> -; Spec (none) -> 75V
- C205: renamed from C401; Mfg_Name (none) -> -; Mfg_PN (none) -> -; Note (none) -> -; Spec (none) -> 10V
- C206: renamed from C406; Mfg_Name (none) -> -; Mfg_PN (none) -> -; Note ceramic, X[57]R -> -; Spec (none) -> 75V X7R
- P202: renamed from P401; value 43045-1000 -> JST PH header; footprint Connectors_Molex:Molex_Microfit3_Header_02x05_Angled_43045-100x -> Connectors_JST:JST_PH_B9B-PH-K_09x2.00mm_Straight; symbol CONN_01X10 -> CONN_01X09; Mfg_Desc (none) -> Through-hole type shrouded header, straight; Mfg_Name (none) -> JST; Mfg_PN (none) -> JST B9B-PH-K-S; Note MicroFit3 2x5 header -> (none)
- P203: renamed from P402; value 43025-1000 -> JST PH housing; symbol CONN_01X10 -> CONN_01X09; Mfg_Desc (none) -> housing, 9-contact; Mfg_Name (none) -> JST; Mfg_PN (none) -> PHR-9; Note MicroFit3 2x5 recept. -> (none)
- Q201: renamed from Q401; Mfg_Name (none) -> Fairchild; Mfg_PN (none) -> BSS138; Note (none) -> -
- R202: renamed from R402; Mfg_Name (none) -> -; Mfg_PN (none) -> -; Note 1%, 50mW -> -; Spec (none) -> 1% 50mW
- R204: renamed from R404; value 2.91k -> 383k; Mfg_Name (none) -> -; Mfg_PN (none) -> -; Note 1%, 50mW -> -; Spec (none) -> 1% 50mW
- U202: renamed from U402; Mfg_Name (none) -> Linear; Mfg_PN (none) -> LTC2991CMS#PBF; Note (none) -> -; Spec (none) -> -
- renumbered SW401 to SW201, SW402 to SW202, SW403 to SW203, U401 to U201, U403 to U203, U404 to U204, W401 to W201, W402 to W202, W403 to W203, W404 to W204, W405 to W205, W406 to W206
Connections:
- net labels added: 12V_SENSE_H, 12V_SENSE_L, 12V_VOUT, 19V_SENSE_H, 19V_SENSE_L, 19V_VOUT, 5V_SENSE_H, 5V_SENSE_L, 5V_VOUT
- wire segments 193 -> 195
Other:
- note added: "Current Sense Resistors\nfull-scale voltage = 0.300 V\nR_sense_max = 0.300/Imax\n5 A = 60mΩ"
- note added: "Power In"
- note removed: "Current Sense Resistors\nfull-scale voltage = 0.300 V\nR_sense_max = 0.300/Imax\n1 A = 300mΩ\n3 A = 100mΩ\n5 A = 60mΩ\n10 A = 30mΩ"
- moved on the sheet: C205, SW201, SW202, SW203, U202

Commit message: LTC3: Replaced DC-DC converters' individual switches with a single switch.
One main power switch now enables all three converters.

Added pin header to each converter's nINHIBIT pin to facilitate manual
control.
Parts:
- removed Q201: BSS138, TO_SOT_Packages_SMD:SOT-23, symbol Q_NMOS_GSD
- removed SW201: SPDT, symbol SPDT
- removed SW202, SW203: SP3T, symbol SP3T
- removed W202, W204, W206: TEST, Measurement_Points:Test_Point_2Pads, symbol TEST
- added D? (x3): D, symbol D
- added P? (x3): PIN_HEAD_1x2, symbol CONN_01X02
- added SW201: SPST, symbol SPST
- P202: footprint Connectors_JST:JST_PH_B9B-PH-K_09x2.00mm_Straight -> Connectors_JST:JST_PH_B2B-PH-K_09x2.00mm_Straight; symbol CONN_01X09 -> CONN_01X02; Mfg_PN JST B9B-PH-K-S -> JST B2B-PH-K-S
- P203: symbol CONN_01X09 -> CONN_01X02; Mfg_PN PHR-9 -> PHR-2
Connections:
- net 12V_ENn: now also Q202.1 (G); no longer P202.4 (P4)
- net 19V_ENn: now also Q203.1 (G); no longer P202.7 (P7)
- net GND: now also P202.2 (P2), P?.2 (P2), P?.2 (P2), P?.2 (P2); no longer P202.9 (P9)
- net at U201.3 (INHIBIT): now also D?.2 (A), P?.1 (P1)
- net at Q203.3 (D), U204.3 (INHIBIT): now also D?.2 (A), P?.1 (P1)
- net at Q202.3 (D), U203.3 (INHIBIT): now also D?.2 (A), P?.1 (P1)
- net at P203.2 (P2): now also SW201.2
- net at P203.1 (P1): now also SW201.1
- removed net +3V3: P202.2 (P2), P202.5 (P5), P202.8 (P8)
- removed net 12V_INHIBIT_FET: P202.3 (P3), Q202.1 (G)
- removed net 19V_INHIBIT_FET: P202.6 (P6), Q203.1 (G)
- net 5V_INHIBIT_FET: no longer names the net of P202.1 (P1)
- net 5V_INHIBIT_FET: now also D?.1 (K), D?.1 (K), D?.1 (K)
Other:
- note added: "Main Power Switch, Front Panel"
- note removed: "Manual Override Switches, Front Panel"
- note removed: "Toggle 5V converter's INHIBIT FET between +3.3V and\nground. Toggle 12V and 19V converters' INHIBIT FET\nbetween the BeagleBone, +3.3V, or ground.\n\nNB: The 5V converter supplies the BeagleBone. We don't\nwant the BB to be able to commit suicide, thus it does\nnot get a connection to the 5V converter's INHIBIT FET."
- moved on the sheet: C205, P201, Q202, Q203, U202

Commit message: LTC3: Modified LTC DC-DC converter schematic.
Added voltage dividers to both sides of LTC299x current sense
resistors.
Parts:
- added R? (x2): 36k, symbol R
- added R? (x4): 10k, symbol R
- added R? (x2): 20k, symbol R
- R201, R203, R205: symbol R4T -> R
Connections:
- net 5V_VOUT is gone; now on net 5V_SENSE_H: C203.1, C204.1, R201.2, U201.6 (V_OUT)
- net +12V: now also R?.1
- net +19V: now also R?.1
- net +5V: now also U202.2 (V2)
- net 12V_SENSE_H: now also R?.1, R?.2; no longer R203.4
- net 12V_SENSE_L: now also R?.1, R?.2; no longer R203.3
- net 12V_VOUT: now also R?.1
- net 19V_SENSE_H: now also R?.1, R?.2; no longer R205.4
- net 19V_SENSE_L: now also R?.1, R?.2; no longer R205.3
- net 19V_VOUT: now also R?.1
- net 5V_SENSE_H: no longer R201.4
- net GND: now also R?.2, R?.2, R?.2, R?.2
- net at D?.1 (K), D?.1 (K), D?.1 (K): no longer P202.1 (P1)
- removed net 5V_SENSE_L: R201.3, U202.2 (V2)
Other:
- moved on the sheet: P201, P202, P203, SW201, W203, W205

Commit message: LTC3: Modified LTC ignition control schematic.
Gave ignition battery ground node a distinctive symbol.
Parts:
- gave numbers to parts that had none: 14
Connections:
- net at P202.1 (P1): now also D201.1 (K), D202.1 (K), D203.1 (K)
