File: ltc3/kicad/ltc/external_triggers.sch (KiCad schematic (older format))
At the start: 42 parts, among them IC801 TLP3542, IC802 TLP3542, IC803 TLP3542, IC804 TLP3542, M801 W28-XQ1A-0.25, M802 W28-XQ1A-0.25, M803 W28-XQ1A-0.25, M804 W28-XQ1A-0.25, P801 43045-1000, P802 43025-1000, P803 43045-0800, P804 43025-0800, P805 43045-0800, P806 43025-0800, P807 1327G6, P808 1327, P809 1327G6, P810 1327, P811 1327G6, P812 1327, P813 1327G6, P814 1327, Q801 PMV45EN, Q802 PMV45EN, Q803 PMV45EN, Q804 PMV45EN, SW801 SP3T, SW802 SP3T, SW803 SP3T, SW804 SP3T

Commit message: LTC3: Split single-board design into two boards.
Separated the charge controller and cell protection circuitry onto its
own board (kicad/charge_controller).  The DC-DC converters,
BeagleBone, external power and triggers, and ignition fire control
circuitry remains together (kicad/ltc).

Both boards have had their schematics updated.  Sub-sheets for
circuitry moved to the other board were removed.  Still more work
remaining, though (e.g., add I2C connectors to Charge Controller
schematic; add battery power connector to LTC board; etc.).

Schematic components were *not* re-annotated to align with new sheet
numbering, as it would screw up the existing layout work (i.e., placed
components would disappear), and that would make us sad engineers.

Both boards have had their PCB layouts converted to four-layer.
Parts:
- M801, M802, M803, M804, P802, P804, P806, P807, P808, P809, P810, P811, P812, P813, P814, SW801, SW802, SW803, SW804: footprint OFF-BOARD -> (none)
Changed lines of the file:
@@
 LIBS:atmel
 LIBS:audio
-LIBS:bbd
 LIBS:brooktre
 LIBS:cmos4000
@@
 LIBS:transistors
 LIBS:ttl_ieee
-LIBS:Launch_Tower_Computer_III-cache
 EELAYER 25 0
 EELAYER END
 $Descr B 17000 11000
 encoding utf-8
-Sheet 8 8
+Sheet 8 6
 Title "LTC3 External Device Triggers"
 Date "2016-05-09"
@@
 EXT_TRG_EN_1
 $Comp
-L GND #PWR801
+L GND #PWR096
 U 1 1 5721FE15
 P 1650 4100
-F 0 "#PWR801" H 1650 4100 30  0001 C CNN
+F 0 "#PWR096" H 1650 4100 30  0001 C CNN
 F 1 "GND" H 1650 4030 30  0001 C CNN
 F 2 "" H 1650 4100 60  0000 C CNN
@@
 $EndComp
 $Comp
-L +5V #PWR803
+L +5V #PWR097
 U 1 1 5721FE44
 P 2450 2250
-F 0 "#PWR803" H 2450 2100 50  0001 C CNN
+F 0 "#PWR097" H 2450 2100 50  0001 C CNN
 F 1 "+5V" H 2450 2390 50  0000 C CNN
 F 2 "" H 2450 2250 60  0000 C CNN
@@
 EXT_TRG_EN_2
 $Comp
-L GND #PWR809
+L GND #PWR098
 U 1 1 5721FE52
 P 6850 4100
-F 0 "#PWR809" H 6850 4100 30  0001 C CNN
+F 0 "#PWR098" H 6850 4100 30  0001 C CNN
 F 1 "GND" H 6850 4030 30  0001 C CNN
 F 2 "" H 6850 4100 60  0000 C CNN
@@
 $EndComp
 $Comp
-L +5V #PWR811
+L +5V #PWR099
 U 1 1 5721FE81
 P 7650 2250
-F 0 "#PWR811" H 7650 2100 50  0001 C CNN
+F 0 "#PWR099" H 7650 2100 50  0001 C CNN
 F 1 "+5V" H 7650 2390 50  0000 C CNN
 F 2 "" H 7650 2250 60  0000 C CNN
@@
 EXT_TRG_EN_3
 $Comp
-L GND #PWR802
+L GND #PWR0100
 U 1 1 5721FE95
 P 1650 10100
-F 0 "#PWR802" H 1650 10100 30  0001 C CNN
+F 0 "#PWR0100" H 1650 10100 30  0001 C CNN
 F 1 "GND" H 1650 10030 30  0001 C CNN
 F 2 "" H 1650 10100 60  0000 C CNN
@@
 $EndComp
 $Comp
-L +5V #PWR804
+L +5V #PWR0101
 U 1 1 5721FEBE
 P 2450 8250
-F 0 "#PWR804" H 2450 8100 50  0001 C CNN
+F 0 "#PWR0101" H 2450 8100 50  0001 C CNN
 F 1 "+5V" H 2450 8390 50  0000 C CNN
 F 2 "" H 2450 8250 60  0000 C CNN
@@
 EXT_TRG_EN_4
 $Comp
-L GND #PWR810
+L GND #PWR0102
 U 1 1 5721FECC
 P 6850 10100
-F 0 "#PWR810" H 6850 10100 30  0001 C CNN
+F 0 "#PWR0102" H 6850 10100 30  0001 C CNN
 F 1 "GND" H 6850 10030 30  0001 C CNN
 F 2 "" H 6850 10100 60  0000 C CNN
@@
 $EndComp
 $Comp
-L +5V #PWR812
+L +5V #PWR0103
 U 1 1 5721FEFB
 P 7650 8250
-F 0 "#PWR812" H 7650 8100 50  0001 C CNN
+F 0 "#PWR0103" H 7650 8100 50  0001 C CNN
 F 1 "+5V" H 7650 8390 50  0000 C CNN
 F 2 "" H 7650 8250 60  0000 C CNN
@@
 F 0 "P804" H 13700 5150 50  0000 L CNN
 F 1 "43025-0800" V 13800 4250 50  0000 L CNN
-F 2 "OFF-BOARD" H 13700 4650 50  0001 C CNN
+F 2 "" H 13700 4650 50  0001 C CNN
 F 3 "" H 13700 4650 50  0000 C CNN
 F 4 "MicroFit3 2x4 recept." V 13900 4650 50  0000 C CNN "Note"
@@
 F 0 "M803" H 15450 5425 50  0000 C CNN
 F 1 "W28-XQ1A-0.25" H 15450 5225 50  0000 C CNN
-F 2 "OFF-BOARD" H 15450 5300 50  0001 C CNN
+F 2 "" H 15450 5300 50  0001 C CNN
 F 3 "" H 15450 5300 50  0000 C CNN
 	1    15450 5300
@@
 F 0 "M804" H 15850 5425 50  0000 C CNN
 F 1 "W28-XQ1A-0.25" H 15850 5225 50  0000 C CNN
-F 2 "OFF-BOARD" H 15850 5300 50  0001 C CNN
+F 2 "" H 15850 5300 50  0001 C CNN
 F 3 "" H 15850 5300 50  0000 C CNN
 	1    15850 5300
@@
 F 0 "M801" H 14650 5425 50  0000 C CNN
 F 1 "W28-XQ1A-0.25" H 14650 5225 50  0000 C CNN
-F 2 "OFF-BOARD" H 14650 5300 50  0001 C CNN
+F 2 "" H 14650 5300 50  0001 C CNN
 F 3 "" H 14650 5300 50  0000 C CNN
 	1    14650 5300
@@
 F 0 "M802" H 15050 5425 50  0000 C CNN
 F 1 "W28-XQ1A-0.25" H 15050 5225 50  0000 C CNN
-F 2 "OFF-BOARD" H 15050 5300 50  0001 C CNN
+F 2 "" H 15050 5300 50  0001 C CNN
 F 3 "" H 15050 5300 50  0000 C CNN
 	1    15050 5300
@@
 Manual Override Switches, Front Panel
 $Comp
-L GND #PWR817
+L GND #PWR0104
 U 1 1 5721FF2F
 P 11800 2200
-F 0 "#PWR817" H 11800 1950 50  0001 C CNN
+F 0 "#PWR0104" H 11800 1950 50  0001 C CNN
 F 1 "GND" H 11808 2026 50  0001 C CNN
 F 2 "" H 11800 2200 50  0000 C CNN
@@
 F 0 "SW801" V 13650 2250 50  0000 R CNN
 F 1 "SP3T" V 13750 2250 50  0000 R CNN
-F 2 "OFF-BOARD" H 13125 2475 50  0001 C CNN
+F 2 "" H 13125 2475 50  0001 C CNN
 F 3 "" H 13125 2475 50  0000 C CNN
 	1    13750 2300
@@
 F 0 "P802" H 13000 2150 50  0000 L CNN
 F 1 "43025-1000" V 13100 1100 50  0000 L CNN
-F 2 "OFF-BOARD" H 13000 1600 50  0001 C CNN
+F 2 "" H 13000 1600 50  0001 C CNN
 F 3 "" H 13000 1600 50  0000 C CNN
 F 4 "MicroFit3 2x5 recept." V 13200 1100 50  0000 L CNN "Note"
@@
 F 0 "SW802" V 14300 2250 50  0000 R CNN
 F 1 "SP3T" V 14400 2250 50  0000 R CNN
-F 2 "OFF-BOARD" H 13775 2475 50  0001 C CNN
+F 2 "" H 13775 2475 50  0001 C CNN
 F 3 "" H 13775 2475 50  0000 C CNN
 	1    14400 2300
@@
 F 0 "SW803" V 14950 2250 50  0000 R CNN
 F 1 "SP3T" V 15050 2250 50  0000 R CNN
-F 2 "OFF-BOARD" H 14425 2475 50  0001 C CNN
+F 2 "" H 14425 2475 50  0001 C CNN
 F 3 "" H 14425 2475 50  0000 C CNN
 	1    15050 2300
@@
 F 0 "SW804" V 15600 2250 50  0000 R CNN
 F 1 "SP3T" V 15700 2250 50  0000 R CNN
-F 2 "OFF-BOARD" H 15075 2475 50  0001 C CNN
+F 2 "" H 15075 2475 50  0001 C CNN
 F 3 "" H 15075 2475 50  0000 C CNN
 	1    15700 2300
@@
 F 0 "P806" H 13950 7850 50  0000 L CNN
 F 1 "43025-0800" V 14050 6950 50  0000 L CNN
-F 2 "OFF-BOARD" H 13950 7350 50  0001 C CNN
+F 2 "" H 13950 7350 50  0001 C CNN
 F 3 "" H 13950 7350 50  0000 C CNN
 F 4 "MicroFit3 2x4 recept." V 14150 7350 50  0000 C CNN "Note"
@@
 $EndComp
 $Comp
-L GND #PWR818
+L GND #PWR0105
 U 1 1 5721FF7E
 P 12850 7850
-F 0 "#PWR818" H 12850 7600 50  0001 C CNN
+F 0 "#PWR0105" H 12850 7600 50  0001 C CNN
 F 1 "GND" H 12858 7677 50  0000 C CNN
 F 2 "" H 12850 7850 50  0000 C CNN
@@
 F 0 "P807" H 14750 8150 50  0000 L CNN
 F 1 "1327G6" H 15000 8150 50  0001 C CNN
-F 2 "OFF-BOARD" H 14650 8150 50  0001 C CNN
+F 2 "" H 14650 8150 50  0001 C CNN
 F 3 "" H 14650 8150 50  0000 C CNN
 	1    14650 8150
@@
 F 0 "P808" H 14900 8150 50  0000 L CNN
 F 1 "1327" H 15100 8150 50  0001 C CNN
-F 2 "OFF-BOARD" H 14800 8150 50  0001 C CNN
+F 2 "" H 14800 8150 50  0001 C CNN
 F 3 "" H 14800 8150 50  0000 C CNN
 	1    14800 8150
@@
 F 0 "P809" H 15150 8150 50  0000 L CNN
 F 1 "1327G6" H 15400 8150 50  0001 C CNN
-F 2 "OFF-BOARD" H 15050 8150 50  0001 C CNN
+F 2 "" H 15050 8150 50  0001 C CNN
 F 3 "" H 15050 8150 50  0000 C CNN
 	1    15050 8150
@@
 F 0 "P810" H 15300 8150 50  0000 L CNN
 F 1 "1327" H 15500 8150 50  0001 C CNN
-F 2 "OFF-BOARD" H 15200 8150 50  0001 C CNN
+F 2 "" H 15200 8150 50  0001 C CNN
 F 3 "" H 15200 8150 50  0000 C CNN
 	1    15200 8150
@@
 F 0 "P811" H 15550 8150 50  0000 L CNN
 F 1 "1327G6" H 15800 8150 50  0001 C CNN
-F 2 "OFF-BOARD" H 15450 8150 50  0001 C CNN
+F 2 "" H 15450 8150 50  0001 C CNN
 F 3 "" H 15450 8150 50  0000 C CNN
 	1    15450 8150
@@
 F 0 "P812" H 15700 8150 50  0000 L CNN
 F 1 "1327" H 15900 8150 50  0001 C CNN
-F 2 "OFF-BOARD" H 15600 8150 50  0001 C CNN
+F 2 "" H 15600 8150 50  0001 C CNN
 F 3 "" H 15600 8150 50  0000 C CNN
 	1    15600 8150
@@
 F 0 "P813" H 15950 8150 50  0000 L CNN
 F 1 "1327G6" H 16200 8150 50  0001 C CNN
-F 2 "OFF-BOARD" H 15850 8150 50  0001 C CNN
+F 2 "" H 15850 8150 50  0001 C CNN
 F 3 "" H 15850 8150 50  0000 C CNN
 	1    15850 8150
@@
 F 0 "P814" H 16100 8150 50  0000 L CNN
 F 1 "1327" H 16300 8150 50  0001 C CNN
-F 2 "OFF-BOARD" H 16000 8150 50  0001 C CNN
+F 2 "" H 16000 8150 50  0001 C CNN
 F 3 "" H 16000 8150 50  0000 C CNN
 	1    16000 8150
@@
 $EndComp
 $Comp
-L GND #PWR806
+L GND #PWR0106
 U 1 1 57255E0A
 P 4750 3350
-F 0 "#PWR806" H 4750 3350 30  0001 C CNN
+F 0 "#PWR0106" H 4750 3350 30  0001 C CNN
 F 1 "GND" H 4750 3280 30  0001 C CNN
 F 2 "" H 4750 3350 60  0000 C CNN
@@
 	4750 2350 4750 2600
 $Comp
-L +5V #PWR805
+L +5V #PWR0107
 U 1 1 57255E12
 P 4750 2350
-F 0 "#PWR805" H 4750 2200 50  0001 C CNN
+F 0 "#PWR0107" H 4750 2200 50  0001 C CNN
 F 1 "+5V" H 4768 2524 50  0000 C CNN
 F 2 "" H 4750 2350 50  0000 C CNN
@@
 $EndComp
 $Comp
-L GND #PWR816
+L GND #PWR0108
 U 1 1 57258DF7
 P 9900 3350
-F 0 "#PWR816" H 9900 3350 30  0001 C CNN
+F 0 "#PWR0108" H 9900 3350 30  0001 C CNN
 F 1 "GND" H 9900 3280 30  0001 C CNN
 F 2 "" H 9900 3350 60  0000 C CNN
@@
 	9900 2350 9900 2600
 $Comp
-L +5V #PWR815
+L +5V #PWR0109
 U 1 1 57258DFF
 P 9900 2350
-F 0 "#PWR815" H 9900 2200 50  0001 C CNN
+F 0 "#PWR0109" H 9900 2200 50  0001 C CNN
 F 1 "+5V" H 9918 2524 50  0000 C CNN
 F 2 "" H 9900 2350 50  0000 C CNN
@@
 $EndComp
 $Comp
-L GND #PWR814
+L GND #PWR0110
 U 1 1 5725D3AE
 P 9850 9300
-F 0 "#PWR814" H 9850 9300 30  0001 C CNN
+F 0 "#PWR0110" H 9850 9300 30  0001 C CNN
 F 1 "GND" H 9850 9230 30  0001 C CNN
 F 2 "" H 9850 9300 60  0000 C CNN
@@
 	9850 8300 9850 8550
 $Comp
-L +5V #PWR813
+L +5V #PWR0111
 U 1 1 5725D3B6
 P 9850 8300
-F 0 "#PWR813" H 9850 8150 50  0001 C CNN
+F 0 "#PWR0111" H 9850 8150 50  0001 C CNN
 F 1 "+5V" H 9868 8474 50  0000 C CNN
 F 2 "" H 9850 8300 50  0000 C CNN
@@
 $EndComp
 $Comp
-L GND #PWR808
+L GND #PWR0112
 U 1 1 5725DD7F
 P 4750 9350
-F 0 "#PWR808" H 4750 9350 30  0001 C CNN
+F 0 "#PWR0112" H 4750 9350 30  0001 C CNN
 F 1 "GND" H 4750 9280 30  0001 C CNN
 F 2 "" H 4750 9350 60  0000 C CNN
@@
 	4750 8350 4750 8600
 $Comp
-L +5V #PWR807
+L +5V #PWR0113
 U 1 1 5725DD87
 P 4750 8350
-F 0 "#PWR807" H 4750 8200 50  0001 C CNN
+F 0 "#PWR0113" H 4750 8200 50  0001 C CNN
 F 1 "+5V" H 4768 8524 50  0000 C CNN
 F 2 "" H 4750 8350 50  0000 C CNN

Commit message: LTC3: Updates to LTC schematic.
1. Cleaned up top-level sheet.
2. Added board-to-board connectors for power, I2C.
3. Miscelleneous component part selection/changes.
Parts:
- removed IC801, IC802, IC803, IC804: TLP3542, Housings_DIP:DIP-6_W7.62mm, symbol TLP3542
- removed M802, M803, M804: W28-XQ1A-0.25, symbol BREAKER_1P
- removed P801: 43045-1000, Connectors_Molex:Molex_Microfit3_Header_02x05_Angled_43045-100x, symbol CONN_01X10
- removed P802: 43025-1000, symbol CONN_01X10
- removed P803, P805: 43045-0800, Connectors_Molex:Molex_Microfit3_Header_02x04_Angled_43045-080x, symbol CONN_01X08
- removed P804, P806: 43025-0800, symbol CONN_01X08
- removed P807, P809, P811, P813: 1327G6, symbol CONN_01X01
- removed P808, P810, P812, P814: 1327, symbol CONN_01X01
- removed Q801, Q802, Q803, Q804: PMV45EN, TO_SOT_Packages_SMD:SOT-23, symbol PMV45EN
- added M602, M603, M604: 250mA, symbol BREAKER_1P
- added P601: JST PH header, Connectors_JST:JST_PH_B9B-PH-K_09x2.00mm_Straight, symbol CONN_01X09
- added P602: JST PH housing, symbol CONN_01X09
- added P603, P605: MicroFit header, Connectors_Molex:Molex_Microfit3_Header_02x04_Angled_43045-080x, symbol CONN_01X08
- added P604, P606: MicroFit recept., symbol CONN_01X08
- added P607, P608, P609, P610, P611, P612, P613, P614: PowerPole, symbol CONN_01X01
- added Q601, Q602, Q603, Q604: PMV45EN, TO_SOT_Packages_SMD:SOT-23, symbol PMV45EN
- added U601, U602, U603, U604: TLP3542, Housings_DIP:DIP-6_W7.62mm, symbol TLP3542
- M601: renamed from M801; value W28-XQ1A-0.25 -> 250mA; Mfg_Name (none) -> TE; Mfg_PN (none) -> W28-XQ1A-0.25; Note (none) -> -; Spec (none) -> -
- renumbered JP801 to JP601, JP802 to JP602, JP803 to JP603, JP804 to JP604, R801 to R601, R802 to R602, R803 to R603, R804 to R604, R805 to R605, R806 to R606, R807 to R607, R808 to R608, SW801 to SW601, SW802 to SW602, SW803 to SW603, SW804 to SW604
Connections:
- net EXT_TRG_1_FET_D: now also P601.1 (P1), Q601.3 (D)
- net EXT_TRG_1_LED_CATH: now also P601.2 (P2), U601.2
- net EXT_TRG_1_OPTO_RELAY: now also P603.2 (P2), U601.6
- net EXT_TRG_2_FET_D: now also P601.3 (P3), Q602.3 (D)
- net EXT_TRG_2_LED_CATH: now also P601.4 (P4), U602.2
- net EXT_TRG_2_OPTO_RELAY: now also P603.4 (P4), U602.6
- net EXT_TRG_3_FET_D: now also P601.5 (P5), Q603.3 (D)
- net EXT_TRG_3_LED_CATH: now also P601.6 (P6), U603.2
- net EXT_TRG_3_OPTO_RELAY: now also P603.6 (P6), U603.6
- net EXT_TRG_4_FET_D: now also P601.7 (P7), Q604.3 (D)
- net EXT_TRG_4_LED_CATH: now also P601.8 (P8), U604.2
- net EXT_TRG_4_OPTO_RELAY: now also P603.8 (P8), U604.6
- net EXT_TRG_EN_1: now also Q601.1 (G)
- net EXT_TRG_EN_2: now also Q602.1 (G)
- net EXT_TRG_EN_3: now also Q603.1 (G)
- net EXT_TRG_EN_4: now also Q604.1 (G)
- net GND: now also P601.9 (P9), P605.2 (P2), P605.4 (P4), P605.6 (P6), P605.8 (P8), Q601.2 (S), Q602.2 (S), Q603.2 (S), Q604.2 (S)
- net at R601.2: now also U601.1
- net at R602.2: now also U602.1
- net at R605.2: now also U603.1
- net at R606.2: now also U604.1
- net at JP601.2: now also P603.1 (P1)
- net at JP602.2: now also P603.3 (P3)
- net at JP604.2: now also P603.5 (P5)
- net at JP603.2: now also P603.7 (P7)
- net at M601.1: now also P604.1 (P1)
- net at M601.2: now also P604.2 (P2)
- net at SW601.1: now also P602.2 (P2)
- net at SW601.3: now also P602.1 (P1)
- net at SW601.4, SW602.4, SW603.4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: now also P602.9 (P9)
- net at SW602.3: now also P602.3 (P3)
- net at SW602.1: now also P602.4 (P4)
- net at SW603.3: now also P602.5 (P5)
- net at SW603.1: now also P602.6 (P6)
- net at SW604.3: now also P602.7 (P7)
- net at SW604.1: now also P602.8 (P8)
- new net: P606.8 (P8), P607.1 (P1)
- new net: P606.7 (P7), P608.1 (P1)
- new net: P606.1 (P1), P614.1 (P1)
- new net: P606.2 (P2), P613.1 (P1)
- new net: P606.3 (P3), P612.1 (P1)
- new net: P606.4 (P4), P611.1 (P1)
- new net: P606.5 (P5), P610.1 (P1)
- new net: P606.6 (P6), P609.1 (P1)
- new net: M602.1, P604.3 (P3)
- new net: M602.2, P604.4 (P4)
- new net: M603.1, P604.5 (P5)
- new net: M603.2, P604.6 (P6)
- new net: M604.1, P604.7 (P7)
- new net: M604.2, P604.8 (P8)
- new net EXT_TRG_1_OUT: P605.1 (P1), U601.4
- new net EXT_TRG_2_OUT: P605.3 (P3), U602.4
- new net EXT_TRG_3_OUT: P605.5 (P5), U603.4
- new net EXT_TRG_4_OUT: P605.7 (P7), U604.4
Other:
- note removed: "12V: 1327 (red)\ngnd: 1327G6 (black)"

Commit message: LTC3: Modified LTC external triggers schematic.
Replaced breakers with 100 ohm current-limiting resistors.
Parts:
- removed M601, M602, M603, M604: 250mA, symbol BREAKER_1P
- removed P603: MicroFit header, Connectors_Molex:Molex_Microfit3_Header_02x04_Angled_43045-080x, symbol CONN_01X08
- removed P604: MicroFit recept., symbol CONN_01X08
- added R? (x4): 100, symbol R
Connections:
- net at JP601.2: now also R?.1
- net at JP602.2: now also R?.1
- net at JP603.2: now also R?.1
- net at JP604.2: now also R?.1
- net EXT_TRG_1_OPTO_RELAY: no longer names the net of U601.6
- net EXT_TRG_1_OPTO_RELAY: now also R?.2
- net EXT_TRG_2_OPTO_RELAY: no longer names the net of U602.6
- net EXT_TRG_2_OPTO_RELAY: now also R?.2
- net EXT_TRG_3_OPTO_RELAY: no longer names the net of U603.6
- net EXT_TRG_3_OPTO_RELAY: now also R?.2
- net EXT_TRG_4_OPTO_RELAY: no longer names the net of U604.6
- net EXT_TRG_4_OPTO_RELAY: now also R?.2
Other:
- note removed: "Circuit Breakers, 250mA x 4, Front Panel"
- moved on the sheet: JP603
