File: ltc3/kicad/ltc/external_power.sch (KiCad schematic (older format))
At the start: 46 parts, among them M501 1A, M502 1A, M503 1A, M504 1A, P501 XH header, P502 XH housing, P503 MicroFit header, P504 MicroFit recept., P505 MicroFit header, P506 MicroFit recept., P507 PowerPole, P508 PowerPole, P509 PowerPole, P510 PowerPole, P511 PowerPole, P512 PowerPole, P513 PowerPole, P514 PowerPole, Q501 PMV45EN, Q502 PMV45EN, Q503 PMV45EN, Q504 PMV45EN, SW501 SP3T, SW502 SP3T, SW503 SP3T, SW504 SP3T, U501 TLP3542, U502 TLP3542, U503 TLP3542, U504 TLP3542

Commit message: LTC3: LTC schematic changes; LTC BOM work.
* Replaced LTC external power and trigger circuits' off-board manual
  override switches with board-mounted tactile momentary switches.
  Simplifies assembly, and should be more than adequate for debugging
  purposes.

* Changed cell protection diodes D1 and D6 from Rohm 1SS355 to ComChip
  CDSU4148.  CDSU4148 is already used on the LTC board, and is higher
  spec than the 1SS355.
Parts:
- removed P501: XH header, -, symbol CONN_01X09
- removed P502: XH housing, -, symbol CONN_01X09
- removed SW501, SW502, SW503, SW504: SP3T, ~, symbol SP3T
- added SW501, SW502, SW503, SW504: MOMENTARY, Buttons_Switches_SMD:SW_SPST_EVQQ2, symbol SW_PUSH_SMALL
- P507, P508, P509, P510, P511, P512, P513, P514: Note - -> OFF-BOARD
Connections:
- net EXT_POW_1_LED_CATH is gone; now on an unnamed net: U501.2
- net EXT_POW_2_LED_CATH is gone; now on an unnamed net: U502.2
- net EXT_POW_3_LED_CATH is gone; now on an unnamed net: U503.2
- net EXT_POW_4_LED_CATH is gone; now on an unnamed net: U504.2
- net GND: now also SW501.2, SW502.2, SW503.2, SW504.2
- net EXT_POW_1_FET_D: no longer names the net of Q501.3 (D)
- net EXT_POW_1_FET_D: now also SW501.1
- net EXT_POW_2_FET_D: no longer names the net of Q502.3 (D)
- net EXT_POW_2_FET_D: now also SW502.1
- net EXT_POW_3_FET_D: no longer names the net of Q503.3 (D)
- net EXT_POW_3_FET_D: now also SW503.1
- net EXT_POW_4_FET_D: no longer names the net of Q504.3 (D)
- net EXT_POW_4_FET_D: now also SW504.1
Other:
- note removed: "Manual Override Switches, Front Panel"
- note removed: "TODO: replace switches w/\nthree-pin jumper header\n(similar to DC-DC converters)?"
- note removed: "Toggle each optoisolator's LED between the FET, disconnected,\nor ground. Use SP3T or SPDT w/ center-NC feature."
- moved on the sheet: C501, C502, C503, C504, M501, M502, M503, M504, P503, P504, P505, P506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

Commit message: LTC3: More work on LTC BOM.
Almost there!
Parts:
- P503, P505: footprint Connectors_Molex:Molex_Microfit3_Header_02x04_Angled_43045-080x -> Connectors_Molex:Molex_Microfit3_Header_02x04_Straight_43045-0828; Mfg_Description - -> 8 pos vertical header; Mfg_PN 43045-0800 -> 43045-0828; Note - -> to front panel
- P504: value MicroFit recept. -> MicroFit connector; Mfg_Description - -> 8 pos connector; Note - -> OFF-BOARD; mates to P503
- P506: value MicroFit recept. -> MicroFit connector; Mfg_Description - -> 8 pos connector; Note - -> OFF-BOARD; mates to P505
Changed lines of the file:
@@
 F 0 "P503" H 12950 4400 50  0000 L CNN
 F 1 "MicroFit header" V 13050 3500 50  0000 L CNN
-F 2 "Connectors_Molex:Molex_Microfit3_Header_02x04_Angled_43045-080x" H 12950 3900 50  0001 C CNN
-F 3 "~" H 12950 3900 50  0001 C CNN
-F 4 "-" H 0   -750 50  0001 C CNN "Mfg_Description"
+F 2 "Connectors_Molex:Molex_Microfit3_Header_02x04_Straight_43045-0828" H 12950 3900 50  0001 C CNN
+F 3 "https://github.com/psas/launch-tower/blob/master/ltc3/doc/datasheets/connectors/Molex-43045-Micro_Fit_3_dual_row_vertical_through_hole_header.pdf" H 12950 3900 50  0001 C CNN
+F 4 "8 pos vertical header" H 0   -750 50  0001 C CNN "Mfg_Description"
 F 5 "Molex" H 12950 3900 60  0001 C CNN "Mfg_Name"
-F 6 "43045-0800" H 12950 3900 60  0001 C CNN "Mfg_PN"
-F 7 "-" V 13150 3500 50  0001 L CNN "Note"
+F 6 "43045-0828" H 12950 3900 60  0001 C CNN "Mfg_PN"
+F 7 "to front panel" V 13150 3500 50  0001 L CNN "Note"
 F 8 "-" H 0   -750 50  0001 C CNN "Spec"
 	1    12950 3900
@@
 P 13700 3900
 F 0 "P504" H 13700 4400 50  0000 L CNN
-F 1 "MicroFit recept." V 13800 3500 50  0000 L CNN
+F 1 "MicroFit connector" V 13800 3500 50  0000 L CNN
 F 2 "~" H 13700 3900 50  0001 C CNN
-F 3 "~" H 13700 3900 50  0001 C CNN
-F 4 "-" H 0   -750 50  0001 C CNN "Mfg_Description"
+F 3 "https://github.com/psas/launch-tower/blob/master/ltc3/doc/datasheets/connectors/Molex-Micro_Fit_3_Family.pdf" H 13700 3900 50  0001 C CNN
+F 4 "8 pos connector" H 0   -750 50  0001 C CNN "Mfg_Description"
 F 5 "Molex" H 13700 3900 60  0001 C CNN "Mfg_Name"
 F 6 "43025-0800" H 13700 3900 60  0001 C CNN "Mfg_PN"
-F 7 "-" V 13900 3900 50  0001 C CNN "Note"
+F 7 "OFF-BOARD; mates to P503" V 13900 3900 50  0001 C CNN "Note"
 F 8 "-" H 0   -750 50  0001 C CNN "Spec"
 	1    13700 3900
@@
 F 0 "P505" H 13200 7100 50  0000 L CNN
 F 1 "MicroFit header" V 13300 6200 50  0000 L CNN
-F 2 "Connectors_Molex:Molex_Microfit3_Header_02x04_Angled_43045-080x" H 13200 6600 50  0001 C CNN
-F 3 "~" H 13200 6600 50  0001 C CNN
-F 4 "-" H 0   -750 50  0001 C CNN "Mfg_Description"
+F 2 "Connectors_Molex:Molex_Microfit3_Header_02x04_Straight_43045-0828" H 13200 6600 50  0001 C CNN
+F 3 "https://github.com/psas/launch-tower/blob/master/ltc3/doc/datasheets/connectors/Molex-43045-Micro_Fit_3_dual_row_vertical_through_hole_header.pdf" H 13200 6600 50  0001 C CNN
+F 4 "8 pos vertical header" H 0   -750 50  0001 C CNN "Mfg_Description"
 F 5 "Molex" H 13200 6600 60  0001 C CNN "Mfg_Name"
-F 6 "43045-0800" H 13200 6600 60  0001 C CNN "Mfg_PN"
-F 7 "-" V 13400 6200 50  0001 L CNN "Note"
+F 6 "43045-0828" H 13200 6600 60  0001 C CNN "Mfg_PN"
+F 7 "to front panel" V 13400 6200 50  0001 L CNN "Note"
 F 8 "-" H 0   -750 50  0001 C CNN "Spec"
 	1    13200 6600
@@
 P 13950 6600
 F 0 "P506" H 13950 7100 50  0000 L CNN
-F 1 "MicroFit recept." V 14050 6200 50  0000 L CNN
+F 1 "MicroFit connector" V 14050 6200 50  0000 L CNN
 F 2 "~" H 13950 6600 50  0001 C CNN
-F 3 "~" H 13950 6600 50  0001 C CNN
-F 4 "-" H 0   -750 50  0001 C CNN "Mfg_Description"
+F 3 "https://github.com/psas/launch-tower/blob/master/ltc3/doc/datasheets/connectors/Molex-Micro_Fit_3_Family.pdf" H 13950 6600 50  0001 C CNN
+F 4 "8 pos connector" H 0   -750 50  0001 C CNN "Mfg_Description"
 F 5 "Molex" H 13950 6600 60  0001 C CNN "Mfg_Name"
 F 6 "43025-0800" H 13950 6600 60  0001 C CNN "Mfg_PN"
-F 7 "-" V 14150 6600 50  0001 C CNN "Note"
+F 7 "OFF-BOARD; mates to P505" V 14150 6600 50  0001 C CNN "Note"
 F 8 "-" H 0   -750 50  0001 C CNN "Spec"
 	1    13950 6600
