File: ltc3/kicad/ltc/LTC3.kicad_pcb (KiCad board)
At the start: 4 copper layers, 202.2 x 150.4 mm, 158 parts, among them IC601 TLP3542, IC701 TLP3542, IC702 TLP3542, IC703 TLP3542, IC704 TLP3542, IC801 TLP3542, IC802 TLP3542, IC803 TLP3542, IC804 TLP3542, J601 RJ45, K601 RELAY_1C, K602 RELAY_1C, P401 43045-1000, P501 BeagleBone_Black_Expansion_He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, P502 BeagleBone_Black_Expansion_He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, P601 BATT-IN, P603 UMBILICAL, P605 43045-0200, P606 S4B-PH-K, P607 43045-0200, P608 43025-0200, P701 43045-1000, P703 43045-0800, P705 43045-0800, P801 43045-1000, P803 43045-0800, P805 43045-0800, Q401 BSS138, Q402 BSS138, Q403 BSS138, Q601 PMV45EN, Q602 PMV45EN, Q603 ZVN4525E6, Q604 ZVN4525E6, Q605 ZVN4525E6, Q701 PMV45EN, Q702 PMV45EN, Q703 PMV45EN, Q704 PMV45EN, Q801 PMV45EN, Q802 PMV45EN, Q803 PMV45EN, Q804 PMV45EN, U401 PTN78020W, U402 LTC2991, U403 PTN78020H, U404 PTN78020H, U501 24C256, U601 CD74HC14, U602 SN65220DBV, U603 741G08

Commit message: LTC3 Layout Work
Did a quick review and made some minor changes to layout.
Routing:
- net +19V: track 281.7 -> 57.4 mm
- added copper zone on Power.Cu, net +19V
Changed lines of the file:
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@@
     (thickness 1.6)
     (drawings 5)
-    (tracks 1283)
+    (tracks 1269)
     (zones 0)
     (modules 158)
@@
     (0 F.Cu mixed)
     (1 Ground.Cu power hide)
-    (2 Power.Cu power hide)
+    (2 Power.Cu power)
     (31 B.Cu mixed hide)
     (32 B.Adhes user)
@@
     (tags "capacitor 0805")
     (attr smd)
-    (fp_text reference C604 (at 2.7432 -0.0381 360) (layer F.SilkS)
+    (fp_text reference C604 (at 2.7432 -0.0381) (layer F.SilkS)
       (effects (font (size 1 1) (thickness 0.15)))
     )
@@
     (tags "resistor 0805")
     (attr smd)
-    (fp_text reference R601 (at 2.4003 -0.5842 360) (layer F.SilkS)
+    (fp_text reference R601 (at 2.4003 -0.5842) (layer F.SilkS)
       (effects (font (size 1 1) (thickness 0.15)))
     )
@@
     (tags "resistor 0805")
     (attr smd)
-    (fp_text reference R616 (at -0.1499 -1.7272 450) (layer F.SilkS)
+    (fp_text reference R616 (at -0.1499 -1.7272 90) (layer F.SilkS)
       (effects (font (size 1 1) (thickness 0.15)))
     )
@@
     (tags "resistor 0805")
     (attr smd)
-    (fp_text reference R610 (at 2.5781 0.1397 360) (layer F.SilkS)
+    (fp_text reference R610 (at 2.5781 0.1397) (layer F.SilkS)
       (effects (font (size 1 1) (thickness 0.15)))
     )
@@
   (segment (start 135.4175 87.122) (end 107.5055 87.122) (width 0.635) (layer F.Cu) (net 20))
   (segment (start 107.5055 87.122) (end 105.2195 89.408) (width 0.635) (layer F.Cu) (net 20))
-  (segment (start 196.2606 152.64) (end 196.2606 148.0006) (width 2.54) (layer Power.Cu) (net 21))
-  (segment (start 97.028 77.216) (end 102.362 71.882) (width 2.54) (layer Power.Cu) (net 21))
-  (segment (start 97.028 124.206) (end 97.028 77.216) (width 2.54) (layer Power.Cu) (net 21))
-  (segment (start 104.902 132.08) (end 97.028 124.206) (width 2.54) (layer Power.Cu) (net 21))
-  (segment (start 104.902 140.208) (end 104.902 132.08) (width 2.54) (layer Power.Cu) (net 21))
-  (segment (start 98.806 146.304) (end 104.902 140.208) (width 2.54) (layer Power.Cu) (net 21))
-  (segment (start 98.806 160.528) (end 98.806 146.304) (width 2.54) (layer Power.Cu) (net 21))
-  (segment (start 110.744 172.466) (end 98.806 160.528) (width 2.54) (layer Power.Cu) (net 21))
-  (segment (start 163.068 172.466) (end 110.744 172.466) (width 2.54) (layer Power.Cu) (net 21))
-  (segment (start 172.72 162.814) (end 163.068 172.466) (width 2.54) (layer Power.Cu) (net 21))
-  (segment (start 172.72 149.098) (end 172.72 162.814) (width 2.54) (layer Power.Cu) (net 21))
-  (segment (start 176.784 145.034) (end 172.72 149.098) (width 2.54) (layer Power.Cu) (net 21))
-  (segment (start 193.294 145.034) (end 176.784 145.034) (width 2.54) (layer Power.Cu) (net 21))
-  (segment (start 196.2606 148.0006) (end 193.294 145.034) (width 2.54) (layer Power.Cu) (net 21))
   (segment (start 102.362 71.882) (end 102.362 76.454) (width 0.635) (layer F.Cu) (net 21))
   (segment (start 125.476 54.356) (end 125.7325 54.6125) (width 0.635) (layer F.Cu) (net 21))
@@
       )
     )
+  )
+  (zone (net 21) (net_name +19V) (layer Power.Cu) (hatch edge 0.508)
+    (connect_pads (clearance 0.508))
+    (min_thickness 0.254)
+    (fill yes (arc_segments 16) (thermal_gap 0.508) (thermal_bridge_width 0.508))
+    (polygon
+      (pts
+        (xy 105.41 162.814) (xy 179.832 162.814) (xy 179.832 148.082) (xy 204.47 148.082) (xy 204.47 173.736)
+        (xy 97.79 173.482) (xy 97.79 67.564) (xy 105.41 67.564) (xy 105.41 162.814)
+      )
+    )

Commit message: LTC3: Modified LTC BOM, schematic.
1. Added footprints for mechanical relays.  (PCB layout already had
   correct footprint; but incorrect annotation.)

2. Created footprint for RJ-45 jack.  This impacts the existing PCB
   layout.
Parts:
- removed P608: 43025-0200, Connectors_Molex:Molex_Microfit3_Header_02x01_Straight_43045-0228
Routing:
- net (no net): track 0.51 -> 0.00 mm
Changed lines of the file:
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@@
-(kicad_pcb (version 4) (host pcbnew "(2016-05-27 BZR 6836, Git 4441a4b)-product")
+(kicad_pcb (version 4) (host pcbnew 4.0.2+dfsg1-stable)
   (general
     (links 371)
     (no_connects 0)
-    (area -107.0207 46.685999 298.828105 197.154001)
+    (area 94.945999 46.5716 298.828107 197.154001)
     (thickness 1.6)
     (drawings 5)
-    (tracks 1269)
+    (tracks 1267)
     (zones 0)
-    (modules 158)
+    (modules 157)
     (nets 117)
   )
@@
       (hpglpenspeed 20)
       (hpglpendiameter 15)
+      (hpglpenoverlay 2)
       (psnegative false)
       (psa4output false)
@@
     (tags "capacitor 0805")
     (attr smd)
-    (fp_text reference C604 (at 2.7432 -0.0381) (layer F.SilkS)
+    (fp_text reference C604 (at 2.7432 -0.0381 360) (layer F.SilkS)
       (effects (font (size 1 1) (thickness 0.15)))
     )
@@
     (tags "resistor 0805")
     (attr smd)
-    (fp_text reference R601 (at 2.4003 -0.5842) (layer F.SilkS)
+    (fp_text reference R601 (at 2.4003 -0.5842 360) (layer F.SilkS)
       (effects (font (size 1 1) (thickness 0.15)))
     )
@@
     (tags "resistor 0805")
     (attr smd)
-    (fp_text reference R616 (at -0.1499 -1.7272 90) (layer F.SilkS)
+    (fp_text reference R616 (at -0.1499 -1.7272 450) (layer F.SilkS)
       (effects (font (size 1 1) (thickness 0.15)))
     )
@@
     (pad "" np_thru_hole circle (at 0 4.32) (size 3.1 3.1) (drill 3.1) (layers *.Cu *.Mask F.SilkS))
   )
-  (module Connectors_Molex:Molex_Microfit3_Header_02x01_Straight_43045-0228 (layer F.Cu)
-    (at -99.06 112.776 90)
-    (descr "Microfit3 Header Straight 02x01 43045-0228")
-    (tags "connector Microfit 02x01 header straight 3mm")
-    (fp_text reference P608 (at 0 5 90) (layer F.SilkS)
-      (effects (font (size 1 1) (thickness 0.15)))
-    )
-    (fp_text value 43025-0200 (at 0 -7 90) (layer F.Fab)
-      (effects (font (size 1 1) (thickness 0.15)))
-    )
-    (fp_line (start 4.5 2.85) (end 4.5 -5.3) (layer F.CrtYd) (width 0.05))
-    (fp_line (start 4.5 2.85) (end -4.5 2.85) (layer F.CrtYd) (width 0.05))
-    (fp_line (start -4.5 2.85) (end -4.5 -5.3) (layer F.CrtYd) (width 0.05))
-    (fp_line (start 4.5 -5.3) (end -4.5 -5.3) (layer F.CrtYd) (width 0.05))
-    (fp_line (start 4.3 2.65) (end 4.3 -5.1) (layer F.SilkS) (width 0.15))
-    (fp_line (start -4.3 2.65) (end -4.3 -5.1) (layer F.SilkS) (width 0.15))
-    (fp_line (start 4.3 2.65) (end -4.3 2.65) (layer F.SilkS) (width 0.15))
-    (fp_line (start 4.3 -5.1) (end -4.3 -5.1) (layer F.SilkS) (width 0.15))
-    (pad "" np_thru_hole circle (at -3 -4 90) (size 1.1 1.1) (drill 1.1) (layers *.Cu *.Mask F.SilkS))
-    (pad 1 thru_hole circle (at 0 0 90) (size 1.6 1.6) (drill 1.1) (layers *.Cu *.Mask F.SilkS))
-    (pad 2 thru_hole circle (at 0 -3 90) (size 1.6 1.6) (drill 1.1) (layers *.Cu *.Mask F.SilkS))
-    (pad "" np_thru_hole circle (at 3 -3.94 90) (size 1.1 1.1) (drill 1.1) (layers *.Cu *.Mask F.SilkS))
-  )
   (module Connectors_Molex:Molex_Microfit3_Header_02x05_Angled_43045-100x (layer F.Cu)
     (at 116.988 179.068)
@@
     (tags "resistor 0805")
     (attr smd)
-    (fp_text reference R610 (at 2.5781 0.1397) (layer F.SilkS)
+    (fp_text reference R610 (at 2.5781 0.1397 360) (layer F.SilkS)
       (effects (font (size 1 1) (thickness 0.15)))
     )
@@
     (descr "Bourns CST0612 Current Sense Resistor")
     (tags "resistor current sense shunt 0612")
-    (fp_text reference R405 (at 3.556 -1.016) (layer F.SilkS)
+    (fp_text reference R405 (at 3.556 -1.016 360) (layer F.SilkS)
       (effects (font (size 1 1) (thickness 0.15)))
     )
@@
     (descr "Bourns CST0612 Current Sense Resistor")
     (tags "resistor current sense shunt 0612")
-    (fp_text reference R403 (at 3.556 -1.016) (layer F.SilkS)
+    (fp_text reference R403 (at 3.556 -1.016 360) (layer F.SilkS)
       (effects (font (size 1 1) (thickness 0.15)))
     )
@@
     (descr "Bourns CST0612 Current Sense Resistor")
     (tags "resistor current sense shunt 0612")
-    (fp_text reference R401 (at 3.556 -1.016) (layer F.SilkS)
+    (fp_text reference R401 (at 3.556 -1.016 360) (layer F.SilkS)
       (effects (font (size 1 1) (thickness 0.15)))
     )
@@
     (effects (font (size 1.5 1.5) (thickness 0.3)))
   )
-  (segment (start 146.812 75.438) (end 146.812 75.692) (width 0.254) (layer F.Cu) (net 0))
-  (segment (start 146.812 75.692) (end 146.812 75.438) (width 0.254) (layer F.Cu) (net 0))
   (segment (start 125.46076 149.926) (end 125.46076 148.57476) (width 0.254) (layer F.Cu) (net 1))
   (via (at 124.714 147.828) (size 1.016) (drill 0.381) (layers F.Cu B.Cu) (net 1))
